File: pcb/eagle/OLM-env-sensor-REVD.sch (EAGLE design)
At the start: 7 parts, among them J1 1X2-3.5MM, U2 AM2302

Commit message: edited env sensor board
Parts:
- removed CON2: (no value), con-harting:CON10L
- added JP1: (no value), SparkFun-Connectors:M03PTH
- added JP3, JP4, JP5: M10", SparkFun-Connectors:M10"
- JP2: value (none) -> M10"; device SparkFun-Connectors:M03PTH -> SparkFun-Connectors:M10"
- renumbered U2 to U1
Connections:
- removed net AIO: CON1.4, CON2.4, J1.2, JP2.2
- removed net DIO1: CON1.2, CON2.2
- removed net DIO2: CON1.9, CON2.9
- removed net DIO3: CON1.7, CON2.7, R1.2, U1.DATA
- removed net VDD: R1.1, U1.VDD
- new net AIO-0: CON1.4, J1.2, JP1.2, JP2.4, JP3.4, JP4.4, JP5.4
- new net DIO-0: CON1.2, JP2.5, JP3.5, JP4.5, JP5.5
- new net DIO-1: CON1.9, JP2.6, JP3.6, JP4.6, JP5.6
- new net DIO-2: CON1.7, JP2.7, JP3.7, JP4.7, JP5.7, R1.2, U1.DATA
- net GND: now also JP1.1, JP2.2, JP3.2, JP4.2, JP5.2; no longer CON2.8, JP2.1
- net MISO: now also JP2.8, JP3.8, JP4.8, JP5.8; no longer CON2.5
- net MOSI: now also JP2.9, JP3.9, JP4.9, JP5.9; no longer CON2.3
- net SCK: now also JP2.10, JP3.10, JP4.10, JP5.10; no longer CON2.1
- net VCC: now also JP2.3, JP3.3, JP4.3, JP5.3, R1.1, U1.VDD; no longer CON2.6
- net VIN: now also JP2.1, JP3.1, JP4.1, JP5.1; no longer CON2.10
Other:
- moved on the sheet: CON1
