File: pcb/eagle/OLM-thermocouple.sch (EAGLE design)
At the start: 18 parts, among them IC1 MAX31855, J1 1X2-3.5MM, J2 1X2-3.5MM, U1 AM2302

Commit message: made some changes
Parts:
- added JP3: M10", SparkFun-Connectors:M10"
- C1: value 10uF -> 0.01µF; device adafruit:C-USC0805K -> microbuilder:CAP_CERAMIC_0805
- C3: value 0.01µF -> 10uF; device microbuilder:CAP_CERAMIC_0805 -> adafruit:C-USC0805K
- D1: value 1n4148 -> 1N4148
- D2: value 1N4148 -> 1n4148
Connections:
- net +3V3: now also C3.1, JP3.3; no longer C1.1
- net AIO-0: now also JP3.4
- net AIO-1: now also D1.C, JP3.5; no longer D2.C
- net CS: now also D1.A, R1.2; no longer D2.A, R2.2
- net DIO-0: now also D2.C, JP3.6; no longer D1.C
- net DIO-1: now also JP3.7
- net GND: now also C3.2, JP3.2; no longer C1.2
- net MISO: now also JP3.8
- net MOSI: now also JP3.9
- net N$4: now also C1.P$1; no longer C3.P$1
- net N$6: now also C1.P$2; no longer C3.P$2
- net SCK: now also D2.A, JP3.10, R2.2; no longer D1.A, R1.2
- net VIN: now also JP3.1
Other:
- moved on the sheet: C1, C2, C3, D1, D2, R1, R2
