File: pcb/eagle/OLM-base-flora.sch (EAGLE design)
At the start: 54 parts, among them CN1 MiniB USB, IC1 ATMEGA32U4-AU, IC2 LP2985-3.3v, IC3 DS1307, IC6 ENC28J60, T1 IRLML2246, U2 USD-SOCKETMICRO-SD-SOCKET-TAO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, X1 32.657k, X2A 25MHz, X2A1 25MHz, X3 8MHz

Commit message: added some details
Connections:
- removed net D0: U2.CS
- removed net SCL: IC3.SCL, RCL.2
- removed net SDA: IC3.SDA, RDA.2
- net D2/SDA: now also IC3.SDA, RDA.2
- net D3/SCL: now also IC3.SCL, RCL.2
Other:
- moved on the sheet: R4, R6, RXLED, TXLED

Commit message: made some changes
Parts:
- removed R10: 330, rcl:R-EU_R0805
- removed X3: 8MHz, adaprog:XTALNX5032
- added JP2, JP3: (no value), SparkFun-Connectors:M08LOCK
- added R5: 1K, adafruit:R-US_R0805
- added X2: 32.657k, crystal:CRYSTALTC26H
- C1: value 0.1u -> 10uF; device rcl:C-EUC0805 -> adafruit:C-USC0805K
- C2, C3: value 18pF -> 10uF
- C7, C8: value 10uF -> 18pF
- C9: value 10uF -> 0.1u; device adafruit:C-USC0805K -> rcl:C-EUC0805
- IC1: value ATMEGA32U4-AU -> LP2985-3.3v; device adaprog:ATMEGA32U4-AU -> adafruit:LP298XS
- IC2: value LP2985-3.3v -> ATMEGA32U4-AU; device adafruit:LP298XS -> adaprog:ATMEGA32U4-AU
- R1: value 22 -> 10K
- R2: value 22 -> 470
- R3: value 470 -> 22
- R4: value 1K -> 22
- R7: value 10K -> 330; device adafruit:R-US_R0805 -> rcl:R-EU_R0805
- X1: value 32.657k -> 8MHz; device crystal:CRYSTALTC26H -> adaprog:XTALNX5032
- renumbered IC6 to IC4, R11 to R8, RN4 to RN1, U2 to U1
Connections:
- removed net AIO: CON1.4, CON2.4, CON3.4, CON4.4
- removed net DIO1: CON1.8, CON2.8, CON3.8, CON4.8
- removed net DIO2: CON1.9, CON2.9, CON3.9, CON4.9
- removed net DIO3: CON1.7, CON2.7, CON3.7, CON4.7
- new net A4/SDA: JP2.8
- new net A5/SCL: JP2.7
- new net D2: JP2.4
- new net D3/PWM: JP2.3
- new net E-CLK: JP2.6
- new net E-INT: JP2.5
- net +3V3: now also C2.1, C3.1, C4.1, C9.1, CON1.6, CON2.6, CON3.6, CON4.6, IC1.VOUT, IC2.AREF, IC2.AVCC, IC2.AVCC1, IC2.UCAP, IC2.VCC, IC2.VCC1, R2.2; no longer C1.1, C6.1, C7.1, C8.1, IC1.AREF, IC1.AVCC, IC1.AVCC1, IC1.UCAP, IC1.VCC, IC1.VCC1, IC2.VOUT, R3.2
- net +5V: now also C1.1, D2.A, IC2.VBUS; no longer C9.1, D1.A, IC1.VBUS
- net A0: now also CON1.4, CON3.4, IC2.PF7(ADC7(TDI); no longer IC1.PF7(ADC7(TDI)
- net A1: now also CON1.2, CON3.2, IC2.PF6(ADC6/TDO); no longer IC1.PF6(ADC6/TDO)
- net A2: now also CON2.4, CON4.4, IC2.PF5(ADC5/TMS); no longer IC1.PF5(ADC5/TMS)
- net A3: now also CON2.2, CON4.2, IC2.PF4(ADC4/TCK); no longer IC1.PF4(ADC4/TCK)
- net A4: now also IC2.PF1(ADC1); no longer IC1.PF1(ADC1)
- net A5: now also IC2.PF0(ADC0); no longer IC1.PF0(ADC0)
- net D0/RX: now also IC2.PD2(INT2/RXD1), JP3.5; no longer IC1.PD2(INT2/RXD1)
- net D1/TX: now also IC2.PD3(INT3/TXD1), JP3.4; no longer IC1.PD3(INT3/TXD1)
- net D2/SDA: now also IC2.PD1(INT1/SDA); no longer IC1.PD1(INT1/SDA)
- net D3/SCL: now also IC2.PD0(INT0/OC0B); no longer IC1.PD0(INT0/OC0B)
- net D4/A6: now also IC2.PD4(ICP1/ADC8); no longer IC1.PD4(ICP1/ADC8)
- net D5*: now also CON1.9, CON3.9, IC2.PC6(OC1A); no longer IC1.PC6(OC1A)
- net D6*/A8: now also IC2.PD7(OC4D/ADC10/T0); no longer IC1.PD7(OC4D/ADC10/T0)
- net D7/AIN0: now also IC2.PE6; no longer IC1.PE6
- net GND: now also CON1.8, CON2.8, CON3.8, CON4.8, IC2.GND1, IC2.GND2, IC2.GND3, IC2.PE2(HWB), IC2.UGND, JP2.1, JP3.6, R5.2; no longer CON1.6, CON2.6, CON3.6, CON4.6, IC1.GND1, IC1.GND2, IC1.GND3, IC1.PE2(HWB), IC1.UGND, R4.2
- net IO10*/A11: now also CON1.7, CON3.7, IC2.PB6(OC1B/OC4B/ADC13); no longer IC1.PB6(OC1B/OC4B/ADC13)
- net IO11*: now also IC2.PB7(OC0A/OC1C/RTS); no longer IC1.PB7(OC0A/OC1C/RTS)
- net IO12*/A7: now also IC2.PD6(T1/OC4D/ADC9); no longer IC1.PD6(T1/OC4D/ADC9)
- net IO13*: now also IC2.PC7(ICP3/CLK0/OC4A); no longer IC1.PC7(ICP3/CLK0/OC4A)
- net IO8/A9: now also CON2.9, CON4.9, IC2.PB4(ADC11); no longer IC1.PB4(ADC11)
- net IO9*/A10: now also CON2.7, CON4.7, IC2.PB5(OC1A/OC4B/ADC12); no longer IC1.PB5(OC1A/OC4B/ADC12)
- net LEDA: now also R7.2; no longer R10.2
- net MISO: now also IC2.PB3(PDO/MISO); no longer IC1.PB3(PDO/MISO)
- net MISO/D12: now also JP3.2
- net MOSI: now also IC2.PB2(PDI/MISO); no longer IC1.PB2(PDI/MISO)
- net MOSI/D11: now also JP3.3
- net N$1: now also R2.1; no longer R3.1
- net N$11: now also R5.1; no longer R4.1
- net N$13: now also R1.1; no longer R7.1
- net N$2: now also R3.1; no longer R2.1
- net N$3: now also IC2.D-, R4.2; no longer IC1.D-, R1.2
- net N$34: now also R7.1; no longer R10.1
- net N$4: now also IC2.D+, R3.2; no longer IC1.D+, R2.2
- net N$47: now also X2.1; no longer X1.1
- net N$5: now also R4.1; no longer R1.1
- net N$50: now also X2.2; no longer X1.2
- net N$54: now also C10.2; no longer C11.2
- net N$6: now also D1.C, R1.2; no longer D2.C, R7.2
- net N$7: now also D1.A; no longer D2.A
- net N$8: now also C7.1, IC2.XTAL1, X1.P$2; no longer C2.1, IC1.XTAL1, X3.P$2
- net N$9: now also C8.1, IC2.XTAL2, X1.P$1; no longer C3.1, IC1.XTAL2, X3.P$1
- net RST: now also IC2./RESET; no longer IC1./RESET
- net RXLED/SS: now also IC2.PB0(SS); no longer IC1.PB0(SS)
- net SCK: now also IC2.PB1(SCK); no longer IC1.PB1(SCK)
- net SCK/D13: now also JP3.1
- net TCT: now also C11.2; no longer C10.2
- net TXLED: now also IC2.PD5(XCK/CTS); no longer IC1.PD5(XCK/CTS)
- net VCC: now also C6.1, D2.C, IC1.EN, IC1.VIN, JP2.2; no longer C4.1, CON1.10, CON2.10, CON3.10, CON4.10, D1.C, IC2.EN, IC2.VIN
- net VIN: now also CON1.10, CON2.10, CON3.10, CON4.10, JP3.7, JP3.8; no longer CON1.2, CON2.2, CON3.2, CON4.2
Other:
- moved on the sheet: C1, C10, C11, C2, C3, C4, C5, C6, C7, C8, C9, CON1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

Commit message: made some changes
Parts:
- removed CON4: (no value), con-harting:CON10L
Connections:
- removed net A4/SDA: JP2.8
- removed net A5/SCL: JP2.7
- removed net D2: JP2.4
- removed net D3/PWM: JP2.3
- removed net D4: IC4.CS
- removed net RESET: IC4.RESET
- net +3V3: no longer CON4.6
- net A0: no longer CON3.4
- net A1: no longer CON3.2
- net A2: no longer CON4.4
- net A3: no longer CON4.2
- net A4: now also CON3.4
- net A5: now also CON3.2
- net D2/SDA: now also JP2.8
- net D3/SCL: now also JP2.7
- net D4/A6: now also IC4.RESET, JP2.4
- net D5*: no longer CON3.9
- net D6*/A8: now also IC4.CS, JP2.3
- net D7/AIN0: now also JP2.2, U1.CS
- net E-CLK: now also IC4.CLKOUT
- net E-INT: now also IC4./INT
- net GND: no longer CON4.8
- net IO10*/A11: no longer CON3.7
- net IO11*: now also CON3.9
- net IO12*/A7: now also CON3.7
- net IO8/A9: no longer CON4.9
- net IO9*/A10: no longer CON4.7
- net MISO: now also JP3.2
- net MISO/D12: no longer CON4.5, JP3.2
- net MOSI: now also JP3.3
- net MOSI/D11: no longer CON4.3, JP3.3
- net SCK: now also JP3.1
- net SCK/D13: no longer CON4.1, JP3.1
- net VCC: now also JP3.8; no longer JP2.2
- net VIN: no longer CON4.10, JP3.8
Other:
- moved on the sheet: R3

Commit message: wrapped up schematic
Other:
- note added: "32u4"
- note added: "Breakout"
- note added: "Connectors"
- note added: "Ethernet"
- note added: "ICSP"
- note added: "Power"
- note added: "RTC"
- note added: "uSD"
- moved on the sheet: BAT1, BATT, BOOT, C1, C10, C11, C2, C3, C4, C5, C6, C7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
