File: pcb/eagle/OLM-base-v.REV-I-SMT.brd (EAGLE design)
At the start: 91.9 x 57.4 mm, 92 parts, among them CN2 DCIN, CN3 MiniB USB, IC1 LP2985-3.3v, IC2 ATMEGA32U4-AU, IC3 ENC28J60, IC4 MCP73871, IC5 DS3231SN, IC6 MCP1703CB, J2 EG1206, T1 IRLML2246, U1 USD-SOCKETMICRO-SD-SOCKET-TAO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, U2 TSL2561, U3 BMP085, U4 AM2302, X1 8MHz, X2A 25MHz

Commit message: olm
Parts:
- removed BATT: 3-9VDC, adafruit:JST-PH-2-SMT-RA
- removed C1, C2, C3, C4, C5, C6: 10uF, adafruit:C0805K
- removed D1: SCHOTTKY, adafruit:SOD-123
- removed IC1: LP2985-3.3v, adafruit:SOT23-5L
- removed ON/OFF: EG1390, adafruit:EG1390
- removed PWR: GREEN, adafruit:CHIPLED_0805
- removed R1: 10K, adafruit:R0805
- removed R2: 470, adafruit:R0805
- removed T1: IRLML2246, zetex:SOT-23
Connections:
- net ADDR renamed VIS-NIR-ADDR
- net INT renamed VIS-NIR-INT
- net N$26 renamed RTC-32KHZ
- net N$27 renamed RTC-INT
- net N$28 renamed RTC-RST
- removed net N$1: PWR.A, R2.1
- removed net N$13: ON/OFF.P2, R1.1, T1.3
- removed net N$24: IC5.16
- removed net N$25: IC5.15
- removed net N$6: D1.C, R1.2, T1.2
- removed net N$7: BATT.1, D1.A
- new net RGB-INT: U$2.5
- net +3V3: no longer C2.1, C3.1, C4.1, IC1.5, R2.2
- net +5V: no longer C1.1
- net D2/SDA: no longer IC2.19
- net D3/SCL: no longer IC2.18
- net GND: no longer BATT.2, C1.2, C2.2, C3.2, C4.2, C5.2, C6.2, IC1.2, ON/OFF.O1, ON/OFF.O2, ON/OFF.P1, ON/OFF.S1, PWR.C
- net SCL: now also IC2.18, IC5.16, U$2.2, U3.P$6
- net SDA: now also IC2.19, IC5.15, U$2.6, U3.P$7
- net VCC: no longer C5.1, C6.1, IC1.1, IC1.3, T1.1

Commit message: added schematic
Parts:
- removed BOOT: SPST_TACT-KMR2, adafruit:KMR2
- removed D6: SCHOTTKY, adafruit:SOD-123
- removed JP8: BATT, microbuilder:1X02_OVAL
- removed L3: 500mA, adafruit:R1206
- added J1: EG1206, adafruit:EG1206
- added R1: 1K, adafruit:R0805
Connections:
- removed net +5V: IC2.7
- removed net 3.3V: C21.1, C22.1, IC6.2
- removed net BATT1: JP8.1
- removed net D2/SDA: JP4.10
- removed net D3/SCL: JP4.9
- removed net N$43: D6.C, J2.2
- removed net VBUS1: CN3.VBUS, L3.1
- net +3V3: now also C21.1, C22.1, IC6.2; no longer IC2.14, IC2.24, IC2.34, IC2.44
- net E-CLK: no longer IC3.3
- net E-INT: no longer IC3.4
- net GND: now also J1.3; no longer BOOT.2, BOOT.4, JP8.2
- net N$35: now also J2.2; no longer D6.A
- net N$39: now also CN3.VBUS; no longer L3.2
- net RST: now also J1.2, R1.1; no longer BOOT.1, BOOT.3
- net SCL: now also JP4.9
- net SDA: now also JP4.10
- net VCC: now also IC2.14, IC2.24, IC2.34, IC2.44, R1.2; no longer C17.1, C18.+, D3.C, D5.C, IC4.P$18, IC4.P$19, JP2.2, R11.2, R12.2, R13.2, R9.2
- net VIN: now also C17.1, C18.+, D3.C, D5.C, IC2.7, IC4.P$18, IC4.P$19, JP2.2, R11.2, R12.2, R13.2

Commit message: added schematic
Parts:
- removed R17: 10k, rcl:0204/7
- added JP6: (no value), SparkFun-Connectors:1X08_LOCK
- added R2: 10K, adafruit:R0805
Connections:
- removed net DIO-1: R17.2, U4.P$2
- net +3V3: now also R2.1; no longer R17.1
- net D4/A6: now also R2.2, U4.P$2; no longer IC3.10
- net E-CLK: now also IC3.3, JP4.7; no longer JP4.8
- net E-INT: now also IC3.4, JP4.8; no longer JP4.7
- net GND: now also JP6.1
- net IO13*: now also JP6.2
- net RGB-INT: now also JP6.3
- net RTC-32KHZ: now also JP6.6
- net RTC-INT: now also JP6.7
- net RTC-RST: now also JP6.8
- net VIS-NIR-ADDR: now also JP6.5
- net VIS-NIR-INT: now also JP6.4
Changed lines of the file:
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@@
 <element name="THERM" library="adafruit" package="0805-THM" value="10K" x="-11.176" y="-119.38"/>
 <element name="U4" library="sensor" package="AM2302" value="AM2302" x="-9.652" y="-151.384"/>
-<element name="R17" library="rcl" package="0204/7" value="10k" x="-12.446" y="-169.418"/>
 <element name="C19" library="resistor" package="C025-024X044" value="0.1µ" x="-14.986" y="-173.736"/>
 <element name="R18" library="adafruit" package="R0805" value="22" x="-7.62" y="-192.024"/>
@@
 <element name="J1" library="adafruit" package="EG1206" value="EG1206" x="-9.398" y="-237.998"/>
 <element name="R1" library="adafruit" package="R0805" value="1K" x="-15.24" y="-243.586"/>
+<element name="R2" library="adafruit" package="R0805" value="10K" x="-15.24" y="-249.174"/>
+<element name="JP6" library="SparkFun-Connectors" package="1X08_LOCK" value="" x="-15.494" y="-265.684"/>
 </elements>
 <signals>
@@
 <contactref element="C22" pad="2"/>
 <contactref element="J1" pad="3"/>
+<contactref element="JP6" pad="1"/>
 <wire x1="-14.898" y1="-215.138" x2="-6.398" y2="-237.998" width="0" layer="19" extent="1-1"/>
 <wire x1="-14.898" y1="-211.074" x2="-14.898" y2="-215.138" width="0" layer="19" extent="1-1"/>
@@
 <wire x1="-13.716" y1="-173.736" x2="-9.83" y2="-178.308" width="0" layer="19" extent="1-1"/>
 <wire x1="-5.842" y1="-165.184" x2="-13.716" y2="-173.736" width="0" layer="19" extent="1-1"/>
+<wire x1="-15.494" y1="-265.557" x2="-6.398" y2="-237.998" width="0" layer="19" extent="1-1"/>
 <wire x1="-8.906" y1="-130.556" x2="-5.842" y2="-165.184" width="0" layer="19" extent="1-1"/>
 <wire x1="-14.24" y1="-130.556" x2="-8.906" y2="-130.556" width="0" layer="19" extent="1-1"/>
@@
 <contactref element="IC6" pad="2"/>
 <contactref element="U4" pad="P$1"/>
-<contactref element="R17" pad="1"/>
+<contactref element="R2" pad="1"/>
 <wire x1="-16.598" y1="-211.074" x2="-16.598" y2="-215.138" width="0" layer="19" extent="1-1"/>
 <wire x1="-13.782" y1="-205.824" x2="-16.598" y2="-211.074" width="0" layer="19" extent="1-1"/>
 <wire x1="-16.256" y1="-173.736" x2="-13.782" y2="-205.824" width="0" layer="19" extent="1-1"/>
-<wire x1="-16.256" y1="-169.418" x2="-16.256" y2="-173.736" width="0" layer="19" extent="1-1"/>
-<wire x1="-13.462" y1="-165.184" x2="-16.256" y2="-169.418" width="0" layer="19" extent="1-1"/>
+<wire x1="-13.462" y1="-165.184" x2="-16.256" y2="-173.736" width="0" layer="19" extent="1-1"/>
+<wire x1="-16.24" y1="-249.174" x2="-16.598" y2="-215.138" width="0" layer="19" extent="1-1"/>
 <wire x1="0.127" y1="-80.8" x2="-13.462" y2="-165.184" width="0" layer="19" extent="1-1"/>
 <wire x1="9.972" y1="-73.152" x2="0.127" y2="-80.8" width="0" layer="19" extent="1-1"/>
@@
 <signal name="IO13*">
 <contactref element="IC2" pad="32"/>
+<contactref element="JP6" pad="2"/>
+<wire x1="-12.954" y1="-265.811" x2="78.444" y2="40.284" width="0" layer="19" extent="1-1"/>
 </signal>
 <signal name="IO10*/A11">
@@
 <signal name="D4/A6">
 <contactref element="IC2" pad="25"/>
-<contactref element="IC3" pad="10"/>
 <contactref element="JP4" pad="6"/>
-<wire x1="52.578" y1="35.352" x2="78.444" y2="34.684" width="0" layer="19" extent="1-1"/>
-<wire x1="27.432" y1="54.991" x2="52.578" y2="35.352" width="0" layer="19" extent="1-1"/>
+<contactref element="U4" pad="P$2"/>
+<contactref element="R2" pad="2"/>
+<wire x1="-14.24" y1="-249.174" x2="-10.922" y2="-165.184" width="0" layer="19" extent="1-1"/>
+<wire x1="78.444" y1="34.684" x2="-10.922" y2="-165.184" width="0" layer="19" extent="1-1"/>
+<wire x1="27.432" y1="54.991" x2="78.444" y2="34.684" width="0" layer="19" extent="1-1"/>
 </signal>
 <signal name="E-CLK">
+<contactref element="IC3" pad="3"/>
+<contactref element="JP4" pad="7"/>
+<wire x1="43.688" y1="35.352" x2="29.972" y2="55.245" width="0" layer="19" extent="1-1"/>
+</signal>
+<signal name="E-INT">
+<contactref element="IC3" pad="4"/>
 <contactref element="JP4" pad="8"/>
-</signal>
-<signal name="E-INT">
-<contactref element="JP4" pad="7"/>
+<wire x1="44.958" y1="35.352" x2="32.512" y2="54.991" width="0" layer="19" extent="1-1"/>
 </signal>
 <signal name="N$10">
@@
 <signal name="VIS-NIR-INT">
 <contactref element="U2" pad="INT"/>
+<contactref element="JP6" pad="4"/>
+<wire x1="3.594" y1="-12.954" x2="-7.874" y2="-265.811" width="0" layer="19" extent="1-1"/>
 </signal>
 <signal name="VIS-NIR-ADDR">
 <contactref element="U2" pad="ADR"/>
+<contactref element="JP6" pad="5"/>
+<wire x1="1.994" y1="-12.954" x2="-5.334" y2="-265.557" width="0" layer="19" extent="1-1"/>
 </signal>
 <signal name="RTC-32KHZ">
 <contactref element="IC5" pad="1"/>
+<contactref element="JP6" pad="6"/>
+<wire x1="-2.794" y1="-265.811" x2="-1.143" y2="-80.8" width="0" layer="19" extent="1-1"/>
 </signal>
 <signal name="RTC-INT">
 <contactref element="IC5" pad="3"/>
+<contactref element="JP6" pad="7"/>
+<wire x1="-0.254" y1="-265.557" x2="1.397" y2="-80.8" width="0" layer="19" extent="1-1"/>
 </signal>
 <signal name="RTC-RST">
 <contactref element="IC5" pad="4"/>
+<contactref element="JP6" pad="8"/>
+<wire x1="2.286" y1="-265.811" x2="2.667" y2="-80.8" width="0" layer="19" extent="1-1"/>
 </signal>
 <signal name="N$20">
@@
 <wire x1="14.97" y1="-91.584" x2="9.636" y2="-110.049" width="0" layer="19" extent="1-1"/>
 </signal>
-<signal name="DIO-1">
-<contactref element="U4" pad="P$2"/>
-<contactref element="R17" pad="2"/>
-<wire x1="-8.636" y1="-169.418" x2="-10.922" y2="-165.184" width="0" layer="19" extent="1-1"/>
-</signal>
 <signal name="N$41">
 <contactref element="CN3" pad="D+"/>
@@
 <signal name="RGB-INT">
 <contactref element="U$2" pad="5"/>
+<contactref element="JP6" pad="3"/>
+<wire x1="-1.016" y1="-12.4745" x2="-10.414" y2="-265.557" width="0" layer="19" extent="1-1"/>
 </signal>
 <signal name="N$1">
