File: pcb/eagle/OLM-base-v.REV-I-SMT.sch (EAGLE design)
At the start: 92 parts, among them CN2 DCIN, CN3 MiniB USB, IC1 LP2985-3.3v, IC2 ATMEGA32U4-AU, IC3 ENC28J60, IC4 MCP73871, IC5 DS3231SN, IC6 MCP1703CB, J2 EG1206, T1 IRLML2246, U1 USD-SOCKETMICRO-SD-SOCKET-TAO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, U2 TSL2561, U3 BMP085, U4 AM2302, X1 8MHz, X2A 25MHz

Commit message: olm
Parts:
- removed BATT: 3-9VDC, adafruit:JST_2PIN-SMT-RA
- removed C1, C2, C3, C4, C5, C6: 10uF, adafruit:C-USC0805K
- removed D1: SCHOTTKY, adafruit:DIODESOD-123
- removed IC1: LP2985-3.3v, adafruit:LP298XS
- removed ON/OFF: EG1390, adafruit:DPDT-EG1390
- removed PWR: GREEN, adafruit:LEDCHIPLED_0805
- removed R1: 10K, adafruit:R-US_R0805
- removed R2: 470, adafruit:R-US_R0805
- removed T1: IRLML2246, zetex:PMOSSOT23
Connections:
- net ADDR renamed VIS-NIR-ADDR
- net INT renamed VIS-NIR-INT
- net N$26 renamed RTC-32KHZ
- net N$27 renamed RTC-INT
- net N$28 renamed RTC-RST
- removed net N$1: PWR.A, R2.1
- removed net N$13: ON/OFF2.P, R1.1, T1.G
- removed net N$24: IC5.SCL
- removed net N$25: IC5.SDA
- removed net N$6: D1.C, R1.2, T1.S
- removed net N$7: BATT.2, D1.A
- new net RGB-INT: U$2.INT
- net +3V3: no longer C2.1, C3.1, C4.1, IC1.VOUT, R2.2
- net +5V: no longer C1.1
- net D2/SDA: no longer IC2.PD1(INT1/SDA)
- net D3/SCL: no longer IC2.PD0(INT0/OC0B)
- net GND: no longer BATT.1, C1.2, C2.2, C3.2, C4.2, C5.2, C6.2, IC1.GND, ON/OFF1.O, ON/OFF1.P, ON/OFF1.S, ON/OFF2.O, PWR.C
- net SCL: now also IC2.PD0(INT0/OC0B), IC5.SCL, U$2.SCL, U3.SCL
- net SDA: now also IC2.PD1(INT1/SDA), IC5.SDA, U$2.SDA, U3.SDA
- net VCC: no longer C5.1, C6.1, IC1.EN, IC1.VIN, T1.D
Other:
- note added: "D2"
- note added: "D3"

Commit message: added schematic
Parts:
- removed BOOT: SPST_TACT-KMR2, adafruit:SPST_TACT-KMR2
- removed D6: SCHOTTKY, adafruit:DIODESOD-123
- removed JP8: BATT, microbuilder:HEADER-1X2
- removed L3: 500mA, adafruit:PTCFUSE-1206
- added J1: EG1206, adafruit:EG1206
- added R1: 1K, adafruit:R-US_R0805
Connections:
- removed net +5V: IC2.VBUS
- removed net 3.3V: C21.1, C22.1, IC6.VO
- removed net BATT1: JP8.1
- removed net D2/SDA: JP4.10
- removed net D3/SCL: JP4.9
- removed net N$43: D6.C, J2.P
- removed net VBUS1: CN3.VBUS, L3.1
- net +3V3: now also C21.1, C22.1, IC6.VO; no longer IC2.AVCC, IC2.AVCC1, IC2.VCC, IC2.VCC1
- net E-CLK: no longer IC3.CLKOUT
- net E-INT: no longer IC3./INT
- net GND: now also J1.S; no longer BOOT.S, BOOT.S1, JP8.2
- net N$35: now also J2.P; no longer D6.A
- net N$39: now also CN3.VBUS; no longer L3.2
- net RST: now also J1.P, R1.1; no longer BOOT.P, BOOT.P1
- net SCL: now also JP4.9
- net SDA: now also JP4.10
- net VCC: now also IC2.AVCC, IC2.AVCC1, IC2.VCC, IC2.VCC1, R1.2; no longer C17.1, C18.+, D3.C, D5.C, IC4.IN1, IC4.IN2, JP2.2, R11.2, R12.2, R13.2, R9.2
- net VIN: now also C17.1, C18.+, D3.C, D5.C, IC2.VBUS, IC4.IN1, IC4.IN2, JP2.2, R11.2, R12.2, R13.2
Other:
- note added: "SENSORS"
- note removed: "non-lipo battery (not controlled)"
- moved on the sheet: BATT1, C11, C12, C13, C14, C16, C17, C18, C19, C20, C21, C22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

Commit message: added schematic
Parts:
- removed R17: 10k, rcl:R-EU_0204/7
- added JP6: (no value), SparkFun-Connectors:M08LOCK
- added R2: 10K, adafruit:R-US_R0805
Connections:
- removed net DIO-1: R17.2, U4.DATA
- net +3V3: now also R2.1; no longer R17.1
- net D4/A6: now also R2.2, U4.DATA; no longer IC3.RESET
- net E-CLK: now also IC3.CLKOUT, JP4.7; no longer JP4.8
- net E-INT: now also IC3./INT, JP4.8; no longer JP4.7
- net GND: now also JP6.1
- net IO13*: now also JP6.2
- net RGB-INT: now also JP6.3
- net RTC-32KHZ: now also JP6.6
- net RTC-INT: now also JP6.7
- net RTC-RST: now also JP6.8
- net VIS-NIR-ADDR: now also JP6.5
- net VIS-NIR-INT: now also JP6.4
