File: pcb/eagle/OLM-base-v.REV-2-SMT.sch (EAGLE design)
At the start: 79 parts, among them CN2 DCIN, CN3 MiniB USB, IC2 ATMEGA32U4-AU, IC3 ENC28J60, IC4 MCP73871, IC5 DS3231SN, IC6 MCP1703CB, J1 EG1206, J2 EG1206, Q1 IRF, U1 USD-SOCKETMICRO-SD-SOCKET-TAO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, U2 TSL2561, U3 BMP085, U4 AM2302, X1 8MHz, X2A 25MHz

Commit message: updated schematic
Parts:
- removed CN2: DCIN, microbuilder:DCBARREL1.3MM
- added B1, B2, B3: (no value), adafruit:31-XX
- added C1: 0.01µF, microbuilder:CAP_CERAMIC_0805
- added C2, C3: 10uF, adafruit:C-USC0805K
- added C4: 1µ, resistor:C-EUC0603
- added C5: 0.1µ, resistor:C-EUC0603
- added C6: 10µ, SparkFun:CAP0603-CAP
- added FB1, FB2: Ferrite, microbuilder:FERRITE_0805
- added HOBBY_IN, SOLAR_IN: (no value), adafruit:JST_2PIN-SMT-RA
- added IC1: MAX31855, adafruit:MAX6675
- added IC8: MCP1703CB, linear:MCP1703CB
- added J3: 1X2-3.5MM, adafruit:1X2-3.5MM
- added JP10, JP11: (no value), SparkFun:M03PTH
- added R17, R20: 2.2k, SparkFun:RESISTOR0402-RES
- added R3, R4: 10K, adafruit:R-US_R0805
Connections:
- removed net GND_BREAK: CN2.GNDBREAK, CN3.GND
- new net A6: B1.P
- new net A7: B2.P
- new net CS: IC1./CS, R4.2
- new net N$22: C4.1, IC8.VI
- new net N$3: FB1.P$1, J3.2
- new net N$4: C1.P$1, FB1.P$2, IC1.T-
- new net N$5: FB2.P$1, J3.1
- new net N$6: C1.P$2, FB2.P$2, IC1.T+
- new net OUT12: JP10.3, R17.1
- new net OUT13: JP11.3, R20.1
- net +3V3: now also C2.1, C3.1, IC1.VCC, R3.1, R4.1
- net D7/AIN0: no longer JP7.5
- net GND: now also B1.S, B2.S, B3.S, C2.2, C3.2, C4.2, C5.2, C6.2, CN3.GND, HOBBY_IN.1, IC1.GND, IC8.GND, JP10.1, JP11.1, SOLAR_IN.1; no longer CN2.GND
- net MISO: now also IC1.DO
- net SCK: now also IC1.SCK, R3.2
- net VCC: no longer JP2.2, JP8.2
- net VIN: now also C5.1, C6.1, IC8.VO, JP10.2, JP11.2, JP2.2, JP8.2, R17.2, R20.2; no longer CN2.PWR
Other:
- note added: "General"
- note added: "LDO to 3.3V"
- note added: "LDO to 5V"
- note added: "Raspberry Pi / Beagle Bone"
- note added: "Thermocouple"
- moved on the sheet: JP3, REA

Commit message: updated design
Parts:
- removed B2, B3: (no value), adafruit:31-XX
- removed CON3: (no value), con-harting:CON10L
- removed J1, J2: EG1206, adafruit:EG1206
- removed JP11: (no value), SparkFun:M03PTH
- removed JP2: (no value), SparkFun:M023.5MM
- removed JP8: (no value), SparkFun:M02JST-PTH-2
- removed Q1: IRF, SparkFun:MOSFET-NCHANNELPTH2
- added BTN: EVQQ2, adafruit:EVQQ2
- added GPS: (no value), SparkFun-Connectors:M04LOCK
- added Q2: (no value), adafruit:MOSFET-NREFLOW
- added S1, S2: 1X2-3.5MM, adafruit:1X2-3.5MM
- added SRV2: (no value), SparkFun:M03PTH
- added SW: SPDT, SparkFun:SWITCH-SPSTSMD2
- renumbered IC1 to THM1, JP10 to SRV1, JP3 to EMBD, JP7 to LCD, U$2 to LUX2, U2 to LUX1
Connections:
- removed net A6: B1.P
- removed net A7: B2.P
- removed net CONTROL: Q1.G, R?2.2
- removed net CS: R4.2, THM1./CS
- removed net OUT12: R17.1, SRV1.3
- removed net OUT13: JP11.3, R20.1
- net +3V3: now also GPS.1; no longer CON3.6
- net A2: now also LCD.4; no longer CON2.4
- net A3: now also LCD.3; no longer CON2.2
- net A4: now also LCD.2; no longer CON3.4, LCD.3
- net A5: now also LCD.1; no longer CON3.2, LCD.4
- net D0/RX: now also GPS.3
- net D1/TX: now also GPS.4
- net D4/A6: now also U1.CS; no longer R2.2, U4.DATA
- net D5*: now also LCD.5; no longer CON1.9
- net D6*/A8: now also CON2.2, R20.1, R4.2, SRV2.3, THM1./CS; no longer IC3.CS, LCD.6
- net D7/AIN0: now also R2.2, U4.DATA; no longer U1.CS
- net GND: now also BTN.P, BTN.P1, GPS.2, Q2.S, SRV2.1; no longer B2.S, B3.S, CON3.8, J1.S, JP11.1, Q1.S
- net HIGH-CURRENT: now also Q2.D, S1.2, S2.2; no longer JP2.1, JP8.1, Q1.D
- net IO10*/A11: now also CON1.9; no longer CON1.7
- net IO11*: now also CON1.7; no longer CON3.9, LCD.2
- net IO12*/A7: now also CON2.4, R17.1, SRV1.3; no longer CON3.7, LCD.1
- net IO13*: now also B1.P, CON2.7
- net IO8/A9: now also IC3.CS, Q2.G, R?2.2
- net IO9*/A10: now also LCD.6; no longer CON2.7
- net MISO: no longer CON3.5
- net MOSI: no longer CON3.3
- net N$22: now also C17.1, C18.+, CN3.VBUS
- net N$35: now also SW.P; no longer J2.P
- net N$44: no longer J2.S
- net RST: now also BTN.S, BTN.S1; no longer J1.P
- net SCK: no longer CON3.1
- net VIN: now also S1.1, S2.1, SRV2.2; no longer C17.1, C18.+, CN3.VBUS, CON3.10, JP11.2, JP2.2, JP8.2
Other:
- note added: "BUTTON"
- note added: "GPS / Radio Breakout"
- note added: "S1"
- note added: "S2"
- note added: "unprotected"
- note removed: "GPS Breakout"
- moved on the sheet: B1, C4, C5, C6, HOBBY_IN, IC8, R20, SOLAR_IN

Commit message: fixed design
Parts:
- removed IC2: ATMEGA32U4-AU, adaprog:ATMEGA32U4-AU
- removed IC5: DS3231SN, comfile:DS3231SN
- removed JP5: STATUS, microbuilder:HEADER-1X2
- removed JP6: (no value), SparkFun-Connectors:M08LOCK
- removed R?2: 10K, adafruit:R-US_M0805
- removed U4: AM2302, sensor:AM2302
- added C23: .01uF, adafruit:C-USC0805
- added IC1: ENC28J60, SparkFun:ENC28J60SO28LONG
- added JP2: ICSP, pinhead:PINHD-2X3
- added JP3: M10LOCK, SparkFun-Connectors:M10LOCK
- added LCD1: (no value), SparkFun-Connectors:M08LOCK
- added LDO3V3: MCP1703CB, linear:MCP1703CB
- added R21: 10K, adafruit:R-US_R0805
- added U2: BMP085, microbuilder:BMP085
- C1: value 0.01µF -> 0.1µ; device microbuilder:CAP_CERAMIC_0805 -> resistor:C-EUC0805
- C10, C9: value 0.1µ -> 18pF; device resistor:C-EUC0805 -> adafruit:C-USC0805
- C11: device adafruit:C-USC0805K -> adafruit:C-USC0805
- C12: value 0.1uF -> 10uF
- C13: value 0.1uF -> 1uF
- C14: value 1.0uF -> 0.1uF; device adafruit:C-USC0805 -> rcl:C-USC0805
- C15: value 0.1uF -> 10uF; device rcl:C-USC0805 -> adafruit:C-USC0805
- C16: value 10uF -> .1uF; device adafruit:C-USC0805K -> adafruit:C-USC0805
- C17: value 10uF/10V -> 1.0uF; device adafruit:C-USC0805K -> adafruit:C-USC0805
- C18: value 4700uF/10V -> 0.1uF; device adafruit:CPOL-USE5-13 -> adafruit:C-USC0805
- C19: value 0.1µ -> .1uF; device resistor:C-EU025-024X044 -> adafruit:C-USC0805
- C2: value 10uF -> 0.1µ; device adafruit:C-USC0805K -> resistor:C-EUC0805
- C20: value 1µ -> 0.1uF; device resistor:C-EUC0603 -> adafruit:C-USC0805
- C21: value 0.1µ -> 10uF; device resistor:C-EUC0603 -> adafruit:C-USC0805
- C22, C6: value 10µ -> 10uF; device SparkFun:CAP0603-CAP -> adafruit:C-USC0805
- C3: value 10uF -> 1uF; device adafruit:C-USC0805K -> adafruit:C-USC0805
- C4: value 1µ -> 4700uF/10V; device resistor:C-EUC0603 -> adafruit:CPOL-USE5-13
- C5: value 0.1µ -> 10uF/10V; device resistor:C-EUC0603 -> adafruit:C-USC0805
- C7: value 18pF -> .1uF; device adafruit:C-USC0805K -> adafruit:C-USC0805
- C8: value 18pF -> 10uF; device adafruit:C-USC0805K -> adafruit:C-USC0805
- IC3: value ENC28J60 -> MCP73871; device SparkFun:ENC28J60SO28LONG -> adafruit:MCP73871
- IC4: value MCP73871 -> ATMEGA32U4-AU; device adafruit:MCP73871 -> adaprog:ATMEGA32U4-AU
- IC6: value MCP1703CB -> DS3231SN; device linear:MCP1703CB -> comfile:DS3231SN
- JP1: value ICSP -> (none); device pinhead:PINHD-2X3 -> SparkFun-Connectors:M08LOCK
- JP4: value M10LOCK -> STATUS; device SparkFun-Connectors:M10LOCK -> microbuilder:HEADER-1X2
- R1: value 1K -> 22
- R11: device adafruit:R-US_R0805 -> adafruit:R-US_M0805
- R14: value 2K -> 10K; device adafruit:R-US_FLIPFLOP -> adafruit:R-US_R0805
- R15: value 100K -> 10K
- R16: value 1K -> 10K; device adafruit:R-US_M0805 -> adafruit:R-US_R0805
- R17: value 2.2k -> 2.2K; device SparkFun:RESISTOR0402-RES -> adafruit:R-US_R0805
- R18: value 22 -> 2.2K
- R19: value 22 -> 10K
- R2: value 10K -> 22
- R20: value 2.2k -> 10K; device SparkFun:RESISTOR0402-RES -> adafruit:R-US_R0805
- R3, R4: value 10K -> 1K
- R6: value 1K -> 270K
- R7: value 10K -> 100K
- R8: value 10K -> 2K; device adafruit:R-US_R0805 -> adafruit:R-US_FLIPFLOP
- R9: value 270K -> 1K
- U3: value BMP085 -> AM2302; device microbuilder:BMP085 -> sensor:AM2302
- renumbered BAT2 to BAT1, BATT1 to BATT, CN3 to USB, HOBBY_IN to HOBBY, IC8 to LDO5V, J3 to THMC, L2 to L1, Q2 to Q1, RT2 to RT1, SOLAR_IN to SOLAR
Connections:
- net +3V3: now also C15.2, C16.2, C17.1, C18.1, C20.1, IC1.VDD, IC1.VDDOSC, IC1.VDDPLL, IC1.VDDRX, IC1.VDDTX, IC4.AREF, IC4.UCAP, IC6.VCC, LCD1.7, LDO3V3.VO, R14.2, R15.2, R16.1, R19.1, R20.1, U2.AVDD, U2.VDD; no longer C12.1, C13.1, C15.1, C2.1, C3.1, IC2.AREF, IC2.UCAP, IC3.VDD, IC3.VDDOSC, IC3.VDDPLL, IC3.VDDRX, IC3.VDDTX, IC5.VCC, IC6.VO, R2.1, R3.1, R4.1, R7.2, R8.2, U3.AVDD, U4.VDD
- net A0: now also IC4.PF7(ADC7(TDI), JP3.2; no longer IC2.PF7(ADC7(TDI), JP4.2
- net A1: now also IC4.PF6(ADC6/TDO); no longer IC2.PF6(ADC6/TDO)
- net A2: now also IC4.PF5(ADC5/TMS), LCD1.4; no longer IC2.PF5(ADC5/TMS)
- net A3: now also IC4.PF4(ADC4/TCK), LCD1.3; no longer IC2.PF4(ADC4/TCK)
- net A4: now also IC4.PF1(ADC1), LCD1.2; no longer IC2.PF1(ADC1)
- net A5: now also IC4.PF0(ADC0), LCD1.1; no longer IC2.PF0(ADC0)
- net BATT: now also C12.1, IC3.VBAT1, IC3.VBAT2, IC3.VBAT3; no longer C16.1, IC4.VBAT1, IC4.VBAT2, IC4.VBAT3
- net D+: now also IC4.D+, R1.2; no longer IC2.D+, R19.2
- net D-: now also IC4.D-, R2.2; no longer IC2.D-, R18.2
- net D0/RX: now also IC4.PD2(INT2/RXD1); no longer IC2.PD2(INT2/RXD1)
- net D1/TX: now also IC4.PD3(INT3/TXD1); no longer IC2.PD3(INT3/TXD1)
- net D4/A6: now also IC4.PD4(ICP1/ADC8), JP3.6; no longer IC2.PD4(ICP1/ADC8), JP4.6
- net D5*: now also IC4.PC6(OC1A), LCD1.5; no longer IC2.PC6(OC1A)
- net D6*/A8: now also IC4.PD7(OC4D/ADC10/T0), JP3.4, R18.1, R19.2; no longer IC2.PD7(OC4D/ADC10/T0), JP4.4, R20.1, R4.2
- net D7/AIN0: now also IC4.PE6, JP3.3, R16.2, U3.DATA; no longer IC2.PE6, JP4.3, R2.2, U4.DATA
- net E-CLK: now also IC1.CLKOUT, JP3.7; no longer IC3.CLKOUT, JP4.7
- net E-INT: now also IC1./INT, JP3.8; no longer IC3./INT, JP4.8
- net GND: now also C1.1, C13.1, C15.1, C16.1, C18.2, C2.1, C3.1, C4.-, C6.1, C7.1, IC1.VSS, IC1.VSSOSC, IC1.VSSPLL, IC1.VSSRX, IC1.VSSTX, IC3.GND1, IC3.GND2, IC3.GND3, IC4.GND, IC4.PE2(HWB), IC4.UGND, IC6.NC1, IC6.NC2, IC6.NC3, IC6.NC4, IC6.NC5, IC6.NC6, IC6.NC7, IC6.NC8, JP1.1, JP2.6, JP3.1, LCD1.8, LDO3V3.GND, R10.1, R12.2, R13.1, R21.1, R7.2, R8.1, U2.GND; no longer C13.2, C15.2, C16.2, C18.-, C2.2, C3.2, C4.2, C6.2, C7.2, C8.2, IC2.GND, IC2.GND1, IC2.GND2, IC2.GND3, IC2.PE2(HWB), IC2.UGND, IC3.VSS, IC3.VSSOSC, IC3.VSSPLL, IC3.VSSRX, IC3.VSSTX, IC5.GND, IC5.NC1, IC5.NC2, IC5.NC3, IC5.NC4, IC5.NC5, IC5.NC6, IC5.NC7, IC5.NC8, JP1.6, JP4.1, JP6.1, R10.2, R14.1, R15.1, R5.2, R6.1, R?2.1, U4.GND
- net IO10*/A11: now also IC4.PB6(OC1B/OC4B/ADC13); no longer IC2.PB6(OC1B/OC4B/ADC13)
- net IO11*: now also IC4.PB7(OC0A/OC1C/RTS); no longer IC2.PB7(OC0A/OC1C/RTS)
- net IO12*/A7: now also IC4.PD6(T1/OC4D/ADC9); no longer IC2.PD6(T1/OC4D/ADC9)
- net IO13*: now also IC4.PC7(ICP3/CLK0/OC4A), JP1.2; no longer IC2.PC7(ICP3/CLK0/OC4A), JP6.2
- net IO8/A9: now also IC1.CS, IC4.PB4(ADC11), R21.2; no longer IC2.PB4(ADC11), IC3.CS, R?2.2
- net IO9*/A10: now also IC4.PB5(OC1A/OC4B/ADC12), LCD1.6; no longer IC2.PB5(OC1A/OC4B/ADC12)
- net MISO: now also IC1.SO, IC4.PB3(PDO/MISO), JP2.1; no longer IC2.PB3(PDO/MISO), IC3.SO, JP1.1
- net MOSI: now also IC1.SI, IC4.PB2(PDI/MISO), JP2.4; no longer IC2.PB2(PDI/MISO), IC3.SI, JP1.4
- net N$1: now also IC6.VBAT; no longer IC5.VBAT
- net N$10: now also C1.2; no longer C9.2
- net N$11: now also R12.1; no longer R5.1
- net N$12: now also R13.2; no longer R6.2
- net N$15: now also IC1.LEDB; no longer IC3.LEDB
- net N$16: now also IC1.VCAP; no longer IC3.VCAP
- net N$17: now also IC1.RBIAS; no longer IC3.RBIAS
- net N$18: now also IC1.OSC2; no longer IC3.OSC2
- net N$19: now also IC1.OSC1; no longer IC3.OSC1
- net N$2: now also IC1.LEDA; no longer IC3.LEDA
- net N$20: now also IC3.VPCC, R6.1, R7.1; no longer IC4.VPCC, R10.1, R9.1
- net N$21: now also IC3./PG; no longer IC4./PG
- net N$22: now also C3.2, C4.+, C5.1; no longer C17.1, C18.+, C4.1
- net N$23: now also IC3.STAT2, JP4.2; no longer IC4.STAT2, JP5.2
- net N$29: now also IC3.STAT1/LBO, JP4.1; no longer IC4.STAT1/LBO, JP5.1
- net N$30: now also R3.1; no longer R11.1
- net N$31: now also R4.1; no longer R12.1
- net N$32: now also R5.1; no longer R13.1
- net N$33: now also IC3.PROG3, R10.2; no longer IC4.PROG3, R15.2
- net N$34: now also IC3.PROG1, R8.2; no longer IC4.PROG1, R14.2
- net N$35: now also IC3.OUT1, IC3.OUT2; no longer IC4.OUT1, IC4.OUT2
- net N$36: now also IC3.THERM, R11.1; no longer IC4.THERM, R16.1
- net N$37: now also R11.2; no longer R16.2
- net N$4: now also C23.1; no longer C1.P$1
- net N$41: now also R1.1; no longer R19.1
- net N$42: now also R2.1; no longer R18.1
- net N$44: now also C13.2, LDO3V3.VI; no longer C20.1, IC6.VI
- net N$6: now also C23.2; no longer C1.P$2
- net N$8: now also C9.2, IC4.XTAL1; no longer C7.1, IC2.XTAL1
- net N$9: now also C10.2, IC4.XTAL2; no longer C8.1, IC2.XTAL2
- net RD+: now also IC1.TPIN+; no longer IC3.TPIN+
- net RD-: now also IC1.TPIN-; no longer IC3.TPIN-
- net RGB-INT: now also JP1.3; no longer JP6.3
- net RST: now also IC1.RESET, IC4./RESET, JP2.5, JP3.5, R9.1; no longer IC2./RESET, IC3.RESET, JP1.5, JP4.5, R1.1
- net RTC-32KHZ: now also IC6.32KHZ, JP1.6; no longer IC5.32KHZ, JP6.6
- net RTC-INT: now also IC6.!INT/SQW, JP1.7; no longer IC5.!INT/SQW, JP6.7
- net RTC-RST: now also IC6.!RST, JP1.8; no longer IC5.!RST, JP6.8
- net RXLED/SS: now also IC4.PB0(SS); no longer IC2.PB0(SS)
- net SCK: now also IC1.SCK, IC4.PB1(SCK), JP2.3, R20.2; no longer IC2.PB1(SCK), IC3.SCK, JP1.3, R3.2
- net SCL: now also IC4.PD0(INT0/OC0B), IC6.SCL, JP3.9, R15.1, U2.SCL; no longer IC2.PD0(INT0/OC0B), IC5.SCL, JP4.9, R8.1, U3.SCL
- net SDA: now also IC4.PD1(INT1/SDA), IC6.SDA, JP3.10, R14.1, U2.SDA; no longer IC2.PD1(INT1/SDA), IC5.SDA, JP4.10, R7.1, U3.SDA
- net TCT: now also C2.2; no longer C10.2
- net TD+: now also IC1.TPOUT+; no longer IC3.TPOUT+
- net TD-: now also IC1.TPOUT-; no longer IC3.TPOUT-
- net TXLED: now also IC4.PD5(XCK/CTS); no longer IC2.PD5(XCK/CTS)
- net VCC: now also IC4.AVCC, IC4.AVCC1, IC4.VCC, IC4.VCC1, R9.2; no longer IC2.AVCC, IC2.AVCC1, IC2.VCC, IC2.VCC1, R1.2
- net VIN: now also C6.2, C7.2, IC3./TE, IC3.CE, IC3.IN1, IC3.IN2, IC3.PROG2, IC3.SEL, IC4.VBUS, R18.2, R3.2, R4.2, R5.2, R6.2; no longer C5.1, C6.1, IC2.VBUS, IC4./TE, IC4.CE, IC4.IN1, IC4.IN2, IC4.PROG2, IC4.SEL, R11.2, R12.2, R13.2, R20.2, R9.2
- net VIS-NIR-ADDR: now also JP1.5; no longer JP6.5
- net VIS-NIR-INT: now also JP1.4; no longer JP6.4
Other:
- note added: "5V Switch"
- note added: "GPS/Radio"
- note added: "LCD (Nokia 5110)"
- note added: "Servos"
- note added: "THMC"
- note removed: "GPS / Radio Breakout"
- note removed: "LCD Nokia 5110"
- note removed: "Servo Breakout"
- note removed: "Switch for CHDK USB triggering via VIN"
- note removed: "needs to be placed close to sensor"
- moved on the sheet: C1, C10, C12, C13, C14, C15, C16, C17, C2, C20, C21, C22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
