File: pcb/eagle/OLM-base-v.REV-3-SMT.sch (EAGLE design)
At the start: 96 parts, among them IC1 ENC28J60, IC3 MCP73871, IC4 ATMEGA32U4-AU, IC6 DS3231SN, U1 USD-SOCKETMICRO-SD-SOCKET-TAO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, U2 BMP085, U3 AM2302, X1 8MHz, X2A 25MHz

Commit message: fixed design
Parts:
- renumbered BATT to BATT3V7
Changed lines of the file:
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@@
 <part name="GND21" library="supply1" deviceset="GND" device=""/>
 <part name="GND24" library="supply1" deviceset="GND" device=""/>
-<part name="BATT" library="adafruit" deviceset="JST_2PIN" device="-SMT-RA"/>
+<part name="BATT3V7" library="adafruit" deviceset="JST_2PIN" device="-SMT-RA"/>
 <part name="GND25" library="supply1" deviceset="GND" device=""/>
 <part name="R8" library="adafruit" deviceset="R-US_" device="FLIPFLOP" value="2K"/>
@@
 <instance part="GND21" gate="1" x="185.42" y="250.19"/>
 <instance part="GND24" gate="1" x="185.42" y="283.21"/>
-<instance part="BATT" gate="G$1" x="205.74" y="275.59" rot="MR180"/>
+<instance part="BATT3V7" gate="G$1" x="205.74" y="275.59" rot="MR180"/>
 <instance part="GND25" gate="1" x="195.58" y="270.51"/>
 <instance part="R8" gate="G$1" x="104.14" y="260.35" rot="R90"/>
@@
 <segment>
 <wire x1="195.58" y1="273.05" x2="203.2" y2="273.05" width="0.1524" layer="91"/>
-<pinref part="BATT" gate="G$1" pin="1"/>
+<pinref part="BATT3V7" gate="G$1" pin="1"/>
 <pinref part="GND25" gate="1" pin="GND"/>
 </segment>
@@
 <junction x="154.94" y="278.13"/>
 <junction x="154.94" y="275.59"/>
-<pinref part="BATT" gate="G$1" pin="2"/>
+<pinref part="BATT3V7" gate="G$1" pin="2"/>
 <pinref part="IC3" gate="G$1" pin="VBAT1"/>
 <pinref part="IC3" gate="G$1" pin="VBAT2"/>

Commit message: more pcb changes
Parts:
- removed CAP1: 10u, resistor:C-EUC0805
- removed IC4: ATMEGA32U4-AU, adaprog:ATMEGA32U4-AU
- removed JP3: M10LOCK, SparkFun-Connectors:M10LOCK
- removed RBS1: 2.32K, rcl:R-EU_R0805
- added C24: 10uF, adafruit:C-USC0805
- added IC2: MCP73871, adafruit:MCP73871
- added JP1: ICSP, pinhead:PINHD-2X3
- added R4: 1K, adafruit:R-US_R0805
- C1: value 0.1µ -> 10u
- C3: value 1uF -> 0.1µ; device adafruit:C-USC0805 -> resistor:C-EUC0805
- C4: value 4700uF/10V -> 1uF; device adafruit:CPOL-USE5-13 -> adafruit:C-USC0805
- C5: value 10uF/10V -> 4700uF/10V; device adafruit:C-USC0805 -> adafruit:CPOL-USE5-13
- C6: value 10uF -> 10uF/10V
- C7: value .1uF -> 10uF
- C8: value 10uF -> .1uF
- IC3: value MCP73871 -> ATMEGA32U4-AU; device adafruit:MCP73871 -> adaprog:ATMEGA32U4-AU
- JP2: value ICSP -> M10LOCK; device pinhead:PINHD-2X3 -> SparkFun-Connectors:M10LOCK
- R1: value 22 -> 2.32K; device adafruit:R-US_R0805 -> rcl:R-EU_R0805
- R17: value 2.2K -> 10K
- R19: value 10K -> 2.2K
- R3: value 1K -> 22
- renumbered BAT1 to BATRTC, BATT3V7 to BATT3V1, CHRG/LBO to CHRG, IC6 to RTC, LDO3V3 to LDO3V1, LUX1 to LUXNIR, LUX2 to LUXRGB, U2 to PRESS, X2A to EXTL
Connections:
- net +3V3: now also IC3.AREF, IC3.UCAP, R17.1, R21.1; no longer IC4.AREF, IC4.UCAP, R16.1, R19.1
- net A0: now also IC3.PF7(ADC7(TDI); no longer IC4.PF7(ADC7(TDI)
- net A1: now also IC3.PF6(ADC6/TDO); no longer IC4.PF6(ADC6/TDO)
- net A2: now also IC3.PF5(ADC5/TMS); no longer IC4.PF5(ADC5/TMS)
- net A3: now also IC3.PF4(ADC4/TCK); no longer IC4.PF4(ADC4/TCK)
- net A4: now also IC3.PF1(ADC1); no longer IC4.PF1(ADC1)
- net A5: now also IC3.PF0(ADC0); no longer IC4.PF0(ADC0)
- net BATT: now also IC2.VBAT1, IC2.VBAT2, IC2.VBAT3; no longer IC3.VBAT1, IC3.VBAT2, IC3.VBAT3
- net D+: now also IC3.D+, R2.2; no longer IC4.D+, R1.2
- net D-: now also IC3.D-, R3.2; no longer IC4.D-, R2.2
- net D0/RX: now also IC3.PD2(INT2/RXD1); no longer IC4.PD2(INT2/RXD1)
- net D1/TX: now also IC3.PD3(INT3/TXD1); no longer IC4.PD3(INT3/TXD1)
- net D4/A6: now also IC3.PD4(ICP1/ADC8); no longer IC4.PD4(ICP1/ADC8)
- net D5*: now also IC3.PC6(OC1A); no longer IC4.PC6(OC1A)
- net D6*/A8: now also IC3.PD7(OC4D/ADC10/T0), R19.1, R20.2; no longer IC4.PD7(OC4D/ADC10/T0), R18.1, R19.2
- net D7/AIN0: now also IC3.PE6, R17.2; no longer IC4.PE6, R16.2
- net GND: now also C1.2, C4.1, C5.-, C6.2, C8.1, IC2.GND1, IC2.GND2, IC2.GND3, IC3.GND, IC3.PE2(HWB), IC3.UGND, JP1.6, JP2.1, R1.1, R16.1; no longer C1.1, C4.-, C5.2, C6.1, CAP1.2, IC4.GND, IC4.GND1, IC4.GND2, IC4.GND3, IC4.PE2(HWB), IC4.UGND, JP2.6, JP3.1, R21.1, RBS1.1
- net IO10*/A11: now also IC3.PB6(OC1B/OC4B/ADC13); no longer IC4.PB6(OC1B/OC4B/ADC13)
- net IO11*: now also IC3.PB7(OC0A/OC1C/RTS); no longer IC4.PB7(OC0A/OC1C/RTS)
- net IO12*/A7: now also IC3.PD6(T1/OC4D/ADC9), R18.1; no longer IC4.PD6(T1/OC4D/ADC9), R17.1
- net IO13*: now also IC3.PC7(ICP3/CLK0/OC4A); no longer IC4.PC7(ICP3/CLK0/OC4A)
- net IO8/A9: now also IC3.PB4(ADC11), R16.2; no longer IC4.PB4(ADC11), R21.2
- net IO9*/A10: now also IC3.PB5(OC1A/OC4B/ADC12); no longer IC4.PB5(OC1A/OC4B/ADC12)
- net MISO: now also IC3.PB3(PDO/MISO), JP1.1; no longer IC4.PB3(PDO/MISO), JP2.1
- net MOSI: now also IC3.PB2(PDI/MISO), JP1.4; no longer IC4.PB2(PDI/MISO), JP2.4
- net N$10: now also C2.2; no longer C1.2
- net N$16: now also C1.1; no longer CAP1.1
- net N$17: now also R1.2; no longer RBS1.2
- net N$20: now also IC2.VPCC; no longer IC3.VPCC
- net N$21: now also IC2./PG; no longer IC3./PG
- net N$22: now also C4.2, C5.+, C6.1; no longer C3.2, C4.+, C5.1
- net N$29: now also IC2.STAT1/LBO; no longer IC3.STAT1/LBO
- net N$30: now also R4.1; no longer R3.1
- net N$33: now also IC2.PROG3; no longer IC3.PROG3
- net N$34: now also IC2.PROG1; no longer IC3.PROG1
- net N$35: now also IC2.OUT1, IC2.OUT2; no longer IC3.OUT1, IC3.OUT2
- net N$36: now also IC2.THERM; no longer IC3.THERM
- net N$41: now also R2.1; no longer R1.1
- net N$42: now also R3.1; no longer R2.1
- net N$8: now also IC3.XTAL1; no longer IC4.XTAL1
- net N$9: now also IC3.XTAL2; no longer IC4.XTAL2
- net RST: now also IC3./RESET, JP1.5; no longer IC4./RESET, JP2.5
- net RXLED/SS: now also IC3.PB0(SS); no longer IC4.PB0(SS)
- net SCK: now also IC3.PB1(SCK), JP1.3, R21.2; no longer IC4.PB1(SCK), JP2.3, R20.2
- net SCL: now also IC3.PD0(INT0/OC0B), JP2.9; no longer IC4.PD0(INT0/OC0B), JP3.9
- net SDA: now also IC3.PD1(INT1/SDA), JP2.10; no longer IC4.PD1(INT1/SDA), JP3.10
- net TCT: now also C3.2; no longer C2.2
- net TXLED: now also IC3.PD5(XCK/CTS); no longer IC4.PD5(XCK/CTS)
- net VCC: now also IC3.AVCC, IC3.AVCC1, IC3.VCC, IC3.VCC1; no longer IC4.AVCC, IC4.AVCC1, IC4.VCC, IC4.VCC1
- net VIN: now also C8.2, IC2./TE, IC2.CE, IC2.IN1, IC2.IN2, IC2.PROG2, IC2.SEL, IC3.VBUS, R19.2, R4.2; no longer C6.2, IC3./TE, IC3.CE, IC3.IN1, IC3.IN2, IC3.PROG2, IC3.SEL, IC4.VBUS, R17.2, R3.2
Other:
- moved on the sheet: C1, C2, C3, C6, C7, C8, R16, R17, R18, R19, R2, R20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

Commit message: updated layout
Parts:
- removed C24: 10uF, adafruit:C-USC0805
- removed U3: AM2302, sensor:AM2302
- added DHT22: (no value), SparkFun-Connectors:M04LOCK
- RT1: device adafruit:R-US_M0805 -> adafruit:R-US_R0805
- renumbered BATT3V1 to BATT3V3, SRV1 to SV1, SRV2 to SV2
Connections:
- net +3V3: now also DHT22.1; no longer U3.VDD
- net D7/AIN0: now also DHT22.2; no longer U3.DATA
- net GND: now also DHT22.4, RT1.2; no longer RT1.1, U3.GND
- net N$37: now also RT1.1; no longer RT1.2
Other:
- moved on the sheet: B1, R12, R13, RT1, RX, TX
