File: pcb/eagle/OpenLux-v2.brd (EAGLE design)
At the start: 100.1 x 73.2 mm, 81 parts, among them IC1 MCP73871, IC2 ATMEGA32U4-AU, U1 USD-SOCKETMICRO-SD-SOCKET-TAO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, U2 XBEE, U3 MLX90614_, X1 8MHz

Commit message: added some schematics
Parts:
- added C18, C19: 0.1uF, adafruit:C0805
- added LUXNIR1: TSL2561, microbuilder:TSL2561_FN@1
- added LUXRGB1: TCS34725, dwbLibrary:DFN-6
- added R20, R21: 10K, adafruit:R0805
- moved C17 4.13 mm to (71.4, 30.0)
- moved U3 4.07 mm to (71.4, 37.1)
- moved JP2 3.59 mm to (85.9, 25.7)
- moved LCD 2.05 mm to (81.8, 27.4)
- moved LUXRGB 2.03 mm to (98.0, 37.8)
- moved LUXNIR 1.78 mm to (97.8, 35.1)
- moved GPS 1.27 mm to (19.1, 49.8)
Connections:
- net +3V3: now also C18.1, C19.1, LUXNIR1.VDD, LUXRGB1.1, R20.2, R21.2
- net GND: now also C18.2, C19.2, LUXNIR1.VSS, LUXRGB1.3
- net RGB-INT: now also LUXRGB1.5
- net SCL: now also LUXNIR1.CLK, LUXRGB1.2, R21.1
- net SDA: now also LUXNIR1.DATA, LUXRGB1.6, R20.1
- net VIS-NIR-ADDR: now also LUXNIR1.ADR
- net VIS-NIR-INT: now also LUXNIR1.INT
