File: pcb/eagle/OLM-REV-5-SMT.brd (EAGLE design)
At the start: 100 x 80 mm, 84 parts, among them CN1 MiniB USB, IC1 ATMEGA32U4-AU, IC3 ENC28J60, SW1 SPDT, U1 MCP73831, U6 MIC5219-3.3, X3 8MHz

Commit message: changes
Parts:
- removed C29, C30, C31, C32: 10uF, adafruit:C0805K
- removed D3: SCHOTTKY, adafruit:SOD-123
- removed DHT22: (no value), SparkFun-Connectors:1X04_LOCK
- removed F3: PTCSMD, SparkFun:PTC-1206
- removed IC3: ENC28J60, SparkFun:SOIC28WLONG
- removed JP1: ICSP, pinhead:2X03
- removed JP14: External Power, SparkFun:1X02
- removed JP2: M10LOCK, SparkFun-Connectors:1X10_LOCK
- removed JP3: (no value), SparkFun:JST-2-SMD
- removed JP6: External Charge, SparkFun:1X02
- removed JP7: External Switch, SparkFun:1X02
- removed L2: Bead, rcl:R0805
- removed R16, R17, R20, R21: 10K, adafruit:R0805
- removed R18: 10K, rcl:R0805
- removed U$1: BMP180, DSSCircuits:LGA7
- removed U6: MIC5219-3.3, SparkFun:SOT23-5
- removed X3: 8MHz, adaprog:NX5032
- added BKOUT: (no value), SparkFun-Connectors:1X08_LOCK
- added BMP1: BMP180, DSSCircuits:LGA7
- added C4: 10uF, resistor:C0805
- added C5: 1uF, resistor:C0805
- added C6: 4.7u, resistor:C0805
- added C7: .1uF, resistor:C0805
- added C8, C9: 18pF, resistor:C0805
- added D2: SCHOTTKY, adafruit:SOD-123
- added DHT1, OLEDSD: (no value), SparkFun-Connectors:1X04_LOCK
- added EXT-CHG: External Charge, SparkFun:1X02
- added EXT-PWR-F: (no value), SparkFun:JST-2-SMD
- added EXT-PWR1: External Power, SparkFun:1X02
- added EXT-SWITCH: External Switch, SparkFun:1X02
- added F1, F2: PTCSMD, SparkFun:PTC-1206
- added IC2: ENC28J60, SparkFun:SOIC28WLONG
- added ICSP: ICSP, pinhead:2X03
- added ISP-PWR: (no value), SparkFun:SJ_2S-TRACE
- added LDO: MIC5219-3.3, SparkFun:SOT23-5
- added LIPO: MCP73831, SparkFun:SOT23-5
- added NORDIC: M04X2, SparkFun-Connectors:2X4
- added OLEDADA: (no value), SparkFun-Connectors:1X05_LOCK
- added R12, R13, R7: 10K, adafruit:R0805
- added R3: 22, adafruit:R0805
- added R8, R9: 4.7k, adafruit:R0805
- added RC: 3.3K, rcl:R0805
- added X1: 8MHz, adaprog:NX5032
- C10: value 4.7u -> 10uF
- C11, C12: value 100nF -> 10uF; device resistor:C0402 -> resistor:C0805
- C13: device adafruit:C0805K -> resistor:C0805
- C14, C15: value 0.1µ -> 10uF
- C16: value 10u -> 100nF
- C17: value 0.1uF -> 100nF; device rcl:C0805 -> resistor:C0805
- C18: value .1uF -> 10uF
- C19: value 1uF -> 10uF; device adafruit:C0805K -> adafruit:C0805
- C2: value 18pF -> 1uF; device adafruit:C0805K -> resistor:C0805
- C20: value 1uF -> .01uF; device adafruit:C0805K -> adafruit:C0805
- C21: value 10uF -> .1uF
- C22: value 10uF -> 0.1uF; device adafruit:C0805 -> rcl:C0805
- C23: value .01uF -> .1uF
- C24, C25: value 10uF -> .1uF; device adafruit:C0805K -> adafruit:C0805
- C26: value .1uF -> 10u; device adafruit:C0805K -> resistor:C0805
- C27, C28: value 10uF -> 0.1µ; device adafruit:C0805K -> resistor:C0805
- C3: value 18pF -> 10uF; device adafruit:C0805K -> resistor:C0805
- L1: value 500mA -> Bead; device adafruit:R1206 -> rcl:R0805
- R1: value 22 -> 10K; device adafruit:R0805 -> rcl:R0805
- R10: value 2.32K -> 10K; device rcl:R0805 -> adafruit:R0805
- R11: value 3.3K -> 10K; device rcl:R0805 -> adafruit:R0805
- R14: value 10K -> 1k
- R15: value 10K -> 2.32K; device adafruit:R0805 -> rcl:R0805
- R4: value 1K -> 470
- R5: value 470 -> 1K
- U1: value MCP73831 -> USD-SOCKETMICRO-SD-SOCKET-TAOBAO; device SparkFun:SOT23-5 -> SparkFunNew:MICRO-SD-SOCKET-TAOBAO
- moved CON1 185.9 mm to (96.3, 52.6), turned to 270 degrees
- moved CON2 180.5 mm to (96.3, 20.1), turned to 270 degrees
- moved C19 162.8 mm to (63.0, 7.11), turned to 90 degrees
- moved B1 155.5 mm to (36.1, 67.6), turned to 180 degrees
- moved C13 155.1 mm to (-94.0, -58.9)
- moved CDR 145.9 mm to (94.0, 36.6), turned to 90 degrees
- moved C16 143.2 mm to (88.9, 2.54)
- moved IC1 138.4 mm to (64.3, 38.9)
- moved C15 138.0 mm to (-94.0, -70.1)
- moved C17 136.1 mm to (88.9, 8.13)
- moved C14 133.8 mm to (-94.0, -64.5)
- moved THM1 132.7 mm to (67.3, 12.7), turned to 270 degrees
- moved C12 131.4 mm to (-94.0, -53.3)
- moved R14 131.2 mm to (40.9, 13.7)
- moved R15 128.7 mm to (40.4, 36.1)
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Connections:
- removed net ANALOG-IO: CDR.1, R14.1
- removed net GND1: B1.2
- removed net IO12*/A7: CON2.4
- removed net IO13*1: B1.1
- removed net SCL1: R16.1
- removed net SDA1: R15.1
- removed net VDD: C12.1, U$1.2
- removed net VDDIO: C11.1, U$1.3
- new net D4/A6: U1.2
- new net IRQ: NORDIC.8
- new net N$1: BKOUT.3
- new net N$6: B1.1, R7.1
- new net RAW1: ISP-PWR.1
- new net SCK1: R14.2
- net +3V3: now also BMP1.2, BMP1.3, C11.1, C12.1, C13.1, C16.1, C19.1, C2.1, C23.1, C25.1, C3.1, DHT1.1, IC2.15, IC2.19, IC2.20, IC2.25, IC2.28, ISP-PWR.2, NORDIC.2, OLEDADA.5, OLEDSD.2, R10.1, R11.1, R12.1, R7.2, R8.2, R9.2, U1.4; no longer C20.1, C27.1, C28.1, C30.1, DHT22.1, IC3.15, IC3.19, IC3.20, IC3.25, IC3.28, JP1.2, R15.2, R16.2, R17.1, R20.1, R21.1, R5.2
- net +5V: now also C10.1, D2.A, F2.2; no longer C31.1, C32.1, D1.A, L1.2
- net 3.3V: now also C4.1, C5.1, C7.1, LDO.5, R4.2; no longer C13.1, C19.1, C26.1, U6.5
- net A2: now also CON2.2, CON2.4, NORDIC.4
- net A3: now also CON2.9
- net A4: now also CON2.7
- net A5: now also OLEDADA.3
- net CHARGE_STAT: now also LIPO.1, RC.2; no longer R11.2, U1.1
- net D6*/A8: now also R11.2; no longer CON2.2, R20.2
- net D7/AIN0: now also DHT1.2, R10.2; no longer DHT22.2, R17.2
- net E-CLK: now also IC2.3; no longer IC3.3
- net E-INT: now also IC2.4; no longer IC3.4
- net GND: now also B1.2, BKOUT.1, BMP1.7, C14.2, C15.2, C23.2, C27.1, C28.1, C4.2, C5.2, C6.2, C7.2, C8.1, C9.1, DHT1.4, EXT-CHG.1, EXT-PWR-F.1, EXT-PWR1.1, IC2.11, IC2.18, IC2.2, IC2.21, IC2.22, ICSP.6, LDO.2, LIPO.2, NORDIC.1, OLEDADA.4, OLEDSD.1, R1.1, R13.2, R14.1, R15.1, R5.2, U1.6, U1.GND1, U1.GND3, U1.P$1, U1.P$2; no longer C14.1, C15.1, C20.2, C27.2, C28.2, C29.2, C30.2, C31.2, C32.2, DHT22.4, IC3.11, IC3.18, IC3.2, IC3.21, IC3.22, JP1.6, JP14.1, JP2.1, JP3.1, JP6.1, R10.1, R14.2, R18.1, R4.2, U$1.7, U1.2, U6.2
- net IO13*: now also BKOUT.2, LCD.6; no longer CON2.7
- net IO8/A9: now also IC2.9; no longer CON2.9, IC3.9
- net IO9*/A10: now also CDR.1, R13.1; no longer LCD.6
- net MISO: now also IC2.6, ICSP.1, NORDIC.7, U1.7; no longer IC3.6, JP1.1
- net MOSI: now also IC2.7, ICSP.4, NORDIC.6, U1.3; no longer IC3.7, JP1.4
- net N$10: now also R4.1; no longer R5.1
- net N$11: now also R5.1; no longer R4.1
- net N$14: now also EXT-SWITCH.2, F1.2; no longer F3.2, JP7.2
- net N$15: now also C27.2; no longer C15.2
- net N$16: now also IC2.26; no longer IC3.26
- net N$17: now also C26.1, IC2.1; no longer C16.1, IC3.1
- net N$18: now also IC2.14, R15.2; no longer IC3.14, R10.2
- net N$19: now also IC2.24; no longer IC3.24
- net N$20: now also IC2.23; no longer IC3.23
- net N$21: now also IC2.27; no longer IC3.27
- net N$24: now also C20.1; no longer C23.1
- net N$26: now also C20.2; no longer C23.2
- net N$3: now also R3.2; no longer R1.2
- net N$30: now also RC.1; no longer R11.1
- net N$31: now also LIPO.5, R1.2; no longer R18.2, U1.5
- net N$33: now also D1.A, EXT-CHG.2; no longer D3.A, JP6.2
- net N$5: now also R3.1; no longer R1.1
- net N$8: now also C8.2, X1.P$2; no longer C2.1, X3.P$2
- net N$9: now also C9.2, X1.P$1; no longer C3.1, X3.P$1
- net RAW: now also EXT-SWITCH.1, LDO.1, LDO.3; no longer JP7.1, U6.1, U6.3
- net RD+: now also IC2.13; no longer IC3.13
- net RD-: now also IC2.12; no longer IC3.12
- net RST: now also IC2.10, ICSP.5; no longer IC3.10, JP1.5
- net RTC-32KHZ: now also BKOUT.4
- net RTC-INT: now also BKOUT.5
- net RTC-RST: now also BKOUT.6
- net SCK: now also IC2.8, ICSP.3, NORDIC.5, R12.2, U1.5; no longer IC3.8, JP1.3, R21.2
- net SCL: now also BKOUT.7, BMP1.5, OLEDADA.2, OLEDSD.4, R8.1; no longer JP2.9, U$1.5
- net SDA: now also BKOUT.8, BMP1.6, OLEDADA.1, OLEDSD.3, R9.1; no longer JP2.10, U$1.6
- net TCT: now also C28.2, L1.1; no longer C14.2, L2.1
- net TD+: now also IC2.17; no longer IC3.17
- net TD-: now also IC2.16; no longer IC3.16
- net VBATT: now also C6.1, EXT-PWR-F.2, EXT-PWR1.2, F1.1, LIPO.3; no longer C10.1, F3.1, JP14.2, JP3.2, U1.3
- net VBUS: now also F2.1; no longer L1.1
- net VCC: now also C14.1, C15.1, D2.C, L1.2, LIPO.4; no longer C25.1, C29.1, D3.C, L2.2, U1.4
Other:
- board size 100 x 80 mm -> 100.1 x 73.2 mm

Commit message: added schematic and board images
Parts:
- removed U1: USD-SOCKETMICRO-SD-SOCKET-TAOBAO, SparkFunNew:MICRO-SD-SOCKET-TAOBAO
- added MICROSD: USD-SOCKETMICRO-SD-SOCKET-TAOBAO, SparkFunNew:MICRO-SD-SOCKET-TAOBAO
- moved C13 178.8 mm to (53.3, 42.4), turned to 180 degrees
- moved C12 178.0 mm to (53.3, 46.5), turned to 180 degrees
- moved C11 177.1 mm to (53.3, 50.5), turned to 180 degrees
- moved C10 176.0 mm to (53.3, 54.1), turned to 180 degrees
- moved C15 157.9 mm to (33.3, 23.4)
- moved C14 146.5 mm to (22.9, 23.9)
- moved PWR1 67.8 mm to (6.10, 18.5), turned to 180 degrees
- moved OLEDADA 37.8 mm to (48.5, 28.2)
- moved LCD 36.0 mm to (48.5, 22.9)
- moved C24 29.4 mm to (20.6, 8.38), turned to 0 degrees
- moved EMBD 28.2 mm to (89.2, 13.2)
- moved C3 25.9 mm to (69.8, 58.2)
- moved BKOUT 23.4 mm to (89.7, 40.6)
- moved C20 20.6 mm to (58.7, 12.7), turned to 90 degrees
- moved C2 20.0 mm to (64.8, 58.2)
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Connections:
- net +3V3: now also MICROSD.4; no longer U1.4
- net D4/A6: now also MICROSD.2; no longer U1.2
- net GND: now also MICROSD.6, MICROSD.GND1, MICROSD.GND3, MICROSD.P$1, MICROSD.P$2; no longer U1.6, U1.GND1, U1.GND3, U1.P$1, U1.P$2
- net MISO: now also MICROSD.7; no longer U1.7
- net MOSI: now also MICROSD.3; no longer U1.3
- net SCK: now also MICROSD.5; no longer U1.5
