File: pcb/eagle/OLM-REV-5-SMT.sch (EAGLE design)
At the start: 109 parts, among them CN1 MiniB USB, IC1 ATMEGA32U4-AU, IC2 LP2985-3.3v, IC3 ENC28J60, IC4 MCP73831, T1 IRLML2246, U2 MIC5219, X3 8MHz

Commit message: added in various lipo options
Parts:
- added C26: 4.7uF, SparkFun:CAP0402-CAP
- added C27: 1uF, SparkFun:CAP0402-CAP
- added C28, C30: 10uF, SparkFun:CAP_POL1206
- added C29: 0.1uF, SparkFun:CAP0402-CAP
- added D4: Yellow, SparkFun:LED0603
- added F3: PTCSMD, SparkFun:PTCSMD
- added JP14: External Power, SparkFun:M02PTH
- added JP3: (no value), SparkFun:M02-JST-2MM-SMT
- added JP6: External Charge, SparkFun:M02PTH
- added JP7: External Switch, SparkFun:M02PTH
- added LED2: Red, SparkFun:LED0603
- added R15, R16: 10K, adafruit:R-US_R0805
- added R18: 470, SparkFun:RESISTOR0402-RES
- added R19: 2K, SparkFun:RESISTOR0402-RES
- added R22: 330, SparkFun:RESISTOR0402-RES
- added S2: Power Switch, SparkFun:SWITCH-SPSTSMD
- added U1: MCP73831, SparkFun:MCP73831
- added U6: MIC5219-3.3, SparkFun:V_REG_LDOSMD
Connections:
- new net 3.3V: C27.1, C28.+, C29.2, R22.2, U6.OUT
- new net CHARGE_STAT: R18.1, U1.STAT
- new net N$14: F3.2, JP7.2, S2.S
- new net N$31: R19.1, U1.PROG
- new net N$32: D4.C, R18.2
- new net N$33: LED2.A, R22.1
- new net SCL1: R16.1
- new net SDA1: R15.1
- new net USB_VCC: C26.1, D4.A, JP6.2, U1.VIN
- new net VBATT: C30.+, F3.1, JP14.2, JP3.2, U1.VBAT
- net +3V3: now also R15.2, R16.2
- net GND: now also C26.2, C27.2, C28.-, C29.1, C30.-, JP14.1, JP3.1, JP6.1, LED2.C, R19.2, U1.VSS, U6.GND
- net RAW: now also JP7.1, S2.P, U6.EN, U6.IN
Other:
- note added: "10K for 100mA charging"
- note added: "2K for 500mA charging"
- note added: "I2C pullups"

Commit message: added stuff
Parts:
- removed 3.3VTAP, 3V3TAP2, D6, GND3TAP, GNDTAP, GNDTAP2, IO10, IO12, IO9, RX, SCL, SDA, TX, VCC2: SEWTAP-2.0IN, adafruit:SEWTAP-2.0IN
- removed BATT: 3-9VDC, adafruit:JST_2PIN-SMT-RA
- removed BND: (no value), wirepad:SMD2
- removed BOOT: SPST_TACT-KMR2, adafruit:SPST_TACT-KMR2
- removed C4, C5, C6, C7, C8, C9: 10uF, adafruit:C-USC0805K
- removed CHG: 0805, led:LEDCHIPLED_0805
- removed D2: SCHOTTKY, adafruit:DIODESOD-123
- removed D4: Yellow, SparkFun:LED0603
- removed F1: 500mA, SparkFun:PTCSMD
- removed F2: PTCSMD, SparkFun:PTCSMD
- removed IC2: LP2985-3.3v, adafruit:LP298XS
- removed IC4: MCP73831, SparkFunNew:MCP73831
- removed JST: (no value), adafruit:JST_2PIN-SMT-RA
- removed L: RED, adafruit:LEDCHIPLED_0805
- removed LED1, LED2: Red, SparkFun:LED0603
- removed ON/OFF: EG1390, adafruit:DPDT-EG1390
- removed PG, PVCC: SEWTAP6, LilyPad-Wearables:SEWTAP611
- removed PWR: GREEN, adafruit:LEDCHIPLED_0805
- removed R12: 3.3K, rcl:R-EU_R0805
- removed R13: 10K, rcl:R-EU_R0805
- removed R19: 2K, SparkFun:RESISTOR0402-RES
- removed R22: 330, SparkFun:RESISTOR0402-RES
- removed R3: 470, adafruit:R-US_R0805
- removed R7, R9: 10K, adafruit:R-US_R0805
- removed R8: 150K, adafruit:R-US_R0805
- removed S2: Power Switch, SparkFun:SWITCH-SPSTSMD
- removed SW: SPDT, SparkFun:SWITCH-SPSTSMD2
- removed T1: IRLML2246, zetex:PMOSSOT23
- removed U$2, U$6: FIDUCIAL, adafruit:FIDUCIAL
- removed U2: MIC5219, SparkFun:V_REG_LDOSMD
- added B1: (no value), adafruit:31-XX
- added C31, C32: 10uF, adafruit:C-USC0805K
- added CHG1: 0805, led:LEDCHIPLED_0805
- added CON1, CON2: (no value), con-harting:CON10L
- added SW1: SPDT, SparkFun:SWITCH-SPSTSMD2
- C1: value 0.1uF -> 4.7u; device SparkFun:CAP0402-CAP -> resistor:C-EUC0805
- C10: value 1uF -> 4.7u; device SparkFun:CAP0402-CAP -> resistor:C-EUC0805
- C13, C28, C30: device SparkFun:CAP_POL1206 -> adafruit:C-USC0805K
- C19: value 10uF -> 1uF; device SparkFun:CAP_POL1206 -> adafruit:C-USC0805K
- C20: value 4.7u -> 1uF; device resistor:C-EUC0805 -> adafruit:C-USC0805K
- C24: value 4.7u -> 10uF; device resistor:C-EUC0805 -> adafruit:C-USC0805K
- C25, C27: value 1uF -> 10uF; device SparkFun:CAP0402-CAP -> adafruit:C-USC0805K
- C26: value 4.7uF -> .1uF; device SparkFun:CAP0402-CAP -> adafruit:C-USC0805K
- C29: value 0.1uF -> 10uF; device SparkFun:CAP0402-CAP -> adafruit:C-USC0805K
- D3: value (none) -> SCHOTTKY; device SparkFun:DIODESOD -> adafruit:DIODESOD-123
- PWR1: value (none) -> GREEN; device wirepad:SMD2 -> adafruit:LEDCHIPLED_0805
- R11: value 1K -> 3.3K; device SparkFun:RESISTOR0402-RES -> rcl:R-EU_R0805
- R18: value 470 -> 10K; device SparkFun:RESISTOR0402-RES -> rcl:R-EU_R0805
- R5: value 1K -> 470
Connections:
- removed net D6*: D6.SEW, IC1.PD7(OC4D/ADC10/T0)
- removed net D7: IC1.PE6, L.A
- removed net IO10*: IC1.PB6(OC1B/OC4B/ADC13), IO10.SEW
- removed net IO12*: IC1.PD6(T1/OC4D/ADC9), IO12.SEW
- removed net IO9*: IC1.PB5(OC1A/OC4B/ADC12), IO9.SEW
- removed net N$1: PWR.A, R3.1
- removed net N$13: ON/OFF2.P, R7.1, T1.G
- removed net N$27: CHG.A, R12.1
- removed net N$28: CHG.C, IC4.STAT
- removed net N$29: IC4.PROG, R13.2
- removed net N$32: D4.C, R18.2
- removed net N$38: LED1.A, R11.1
- removed net N$6: D2.C, R7.2, T1.S
- removed net N$7: BATT.2, D2.A
- removed net PC6: IC1.PC6(OC1A)
- removed net PC7: IC1.PC7(ICP3/CLK0/OC4A)
- removed net PD0: IC1.PD0(INT0/OC0B), SCL.SEW
- removed net PD1: IC1.PD1(INT1/SDA), SDA.SEW
- removed net USB_VCC: C26.1, D4.A, JP6.2, U1.VIN
- removed net UVCC: F1.1
- removed net VBAT: IC4.VBAT, JST.2, SW.P
- removed net VPP: BTN.S, BTN.S1
- new net A0: CON1.4
- new net A1: CON1.2
- new net GND1: B1.S
- new net IO10*/A11: CON1.9
- new net IO11*: CON1.7
- new net IO12*/A7: CON2.4
- new net IO13*: CON2.7
- new net IO13*1: B1.P
- net +3V3: now also C20.1, C24.1, C27.1, C28.1, C30.1, CON1.6, CON2.6, JP1.2, R5.2; no longer 3.3VTAP.SEW, 3V3TAP2.SEW, C25.1, C6.1, C7.1, C8.1, IC2.VOUT, R3.2
- net +5V: now also C31.1, C32.1; no longer C9.1
- net 3.3V: now also C13.1, C19.1, C26.1; no longer C27.1, C28.+, C29.2, R22.2
- net A5: no longer IC1.PF0(ADC0), R8.2, R9.1
- net CHARGE_STAT: now also R11.2; no longer R18.1
- net D0/RX: no longer IC1.PD2(INT2/RXD1), RX.SEW
- net D1/TX: no longer IC1.PD3(INT3/TXD1), TX.SEW
- net D6*/A8: now also CON2.2
- net GND: now also C1.2, C13.2, C19.2, C28.2, C29.2, C30.2, C31.2, C32.2, CON1.8, CON2.8, PWR1.C, R18.1; no longer BATT.1, BND.P, BOOT.S, BOOT.S1, C1.1, C13.-, C19.-, C28.-, C29.1, C30.-, C4.2, C5.2, C6.2, C7.2, C8.2, C9.2, GND3TAP.SEW, GNDTAP.SEW, GNDTAP2.SEW, IC1.PE2(HWB), IC2.GND, IC4.VSS, JST.1, LED1.C, LED2.C, ON/OFF1.O, ON/OFF1.P, ON/OFF1.S, ON/OFF2.O, PG.1, PWR.C, R13.1, R19.2, R5.2, R9.2, U2.GND
- net IO8/A9: now also CON2.9
- net MISO: now also CON1.5, CON2.5; no longer IC1.PB3(PDO/MISO)
- net MOSI: now also CON1.3, CON2.3; no longer IC1.PB2(PDI/MISO)
- net N$10: now also PWR1.A; no longer L.C
- net N$14: now also SW1.P; no longer S2.S
- net N$30: now also CHG1.C, R11.1; no longer D3.A, F1.2
- net N$31: now also R18.2; no longer R19.1
- net N$33: now also D3.A, JP6.2; no longer LED2.A, R22.1
- net RAW: now also SW1.O; no longer C19.+, D3.C, S2.P, U2.EN, U2.IN
- net RST: now also BTN.S, BTN.S1; no longer BOOT.P, BOOT.P1
- net RXLED/SS: no longer IC1.PB0(SS)
- net SCK: now also CON1.1, CON2.1; no longer IC1.PB1(SCK)
- net TXLED: no longer IC1.PD5(XCK/CTS)
- net VBATT: now also C10.1; no longer C30.+
- net VBUS: no longer F2.1
- net VCC: now also C1.1, C25.1, C29.1, CHG1.A, D3.C, U1.VIN; no longer C1.2, C10.1, C13.+, C4.1, C5.1, IC2.EN, IC2.VIN, R11.2, R8.1, T1.D, U2.OUT, VCC2.SEW
- net VDD: no longer C20.1, PVCC.1, PWR1.P, SW.O
- net VIN: now also CON1.10, CON2.10; no longer C24.1, F2.2, IC4.VIN, R12.2
Other:
- note added: "BUTTON"
- note added: "Bypassing"
- note added: "D2"
- note added: "D3"
- note added: "Photocell"
- note added: "need to bring up to 3v3?"
- note added: "power circuit from Fio"
- note removed: "Board is marked with combination of"
- note removed: "Buttons"
- note removed: "Lipo Controller"
- note removed: "VCC = 5V or 3.3V Output"
- note removed: "resonator frequency and regulator voltage."
- moved on the sheet: BTN, C1, C10, C14, C15, C16, C20, C24, C25, C26, C27, C29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

Commit message: updated schematic
Parts:
- removed B1: (no value), adafruit:31-XX
- removed C32: 10uF, adafruit:C-USC0805K
- removed JP2: M10LOCK, SparkFun-Connectors:M10LOCK
- removed L1: 500mA, adafruit:PTCFUSE-1206
- added B2: (no value), adafruit:31-XX
- added BKOUT: (no value), SparkFun-Connectors:M08LOCK
- added C4: .1uF, adafruit:C-USC0805
- added F1: PTCSMD, SparkFun:PTCSMD
- added ISP-PWR: SOLDERJUMPERTRACE, SparkFun:SOLDERJUMPERTRACE
- added NORDIC: M04X2, SparkFun-Connectors:M04X2
- added OLEDADA: (no value), SparkFun-Connectors:M05LOCK
- added OLEDSD: (no value), SparkFun-Connectors:M04LOCK
- added R3: 1K, adafruit:R-US_R0805
- added R7: 1k, adafruit:R-US_R0805
- added U2: USD-SOCKETMICRO-SD-SOCKET-TAOBAO, SparkFunNew:USD-SOCKETMICRO-SD-SOCKET-TAOBAO
- R6: value 1K -> 10K
- renumbered JP1 to ICSP, JP14 to EXT-PWR1, JP3 to EXT-PWR-F, JP6 to EXT-CHG, JP7 to EXT-SWITCH
Connections:
- removed net ANALOG-IO: CDR.1, R14.1
- removed net GND1: B1.S
- removed net IO12*/A7: CON2.4
- removed net IO13*1: B1.P
- removed net SCL1: R16.1
- removed net SDA1: R15.1
- new net D4/A6: U2.CS
- new net IRQ: NORDIC.8
- new net N$1: BKOUT.3
- new net N$6: B2.P, R6.1
- new net RAW1: ISP-PWR.1
- new net SCK1: R7.2
- net +3V3: now also C4.1, ISP-PWR.2, NORDIC.2, OLEDADA.5, OLEDSD.2, R6.2, U2.VCC; no longer ICSP.2
- net +5V: now also F1.2; no longer C32.1, L1.2
- net A2: now also CON2.2, CON2.4, NORDIC.4
- net A3: now also CON2.9
- net A4: now also CON2.7
- net A5: now also OLEDADA.3
- net D6*/A8: no longer CON2.2
- net GND: now also B2.S, BKOUT.1, C4.2, NORDIC.1, OLEDADA.4, OLEDSD.1, R3.1, R7.1, U2.GND, U2.SHIELD@1, U2.SHIELD@2, U2.SHIELD@3, U2.SHIELD@4; no longer C32.2, JP2.1, R6.1
- net IO13*: now also BKOUT.2, LCD.6; no longer CON2.7
- net IO8/A9: no longer CON2.9
- net IO9*/A10: now also CDR.1, R14.1; no longer LCD.6
- net MISO: now also NORDIC.7, U2.DO
- net MOSI: now also NORDIC.6, U2.DI
- net N$12: now also R3.2; no longer R6.2
- net RTC-32KHZ: now also BKOUT.4
- net RTC-INT: now also BKOUT.5
- net RTC-RST: now also BKOUT.6
- net SCK: now also NORDIC.5, U2.SCK
- net SCL: now also BKOUT.7, OLEDADA.2, OLEDSD.4, R16.1; no longer JP2.9
- net SDA: now also BKOUT.8, OLEDADA.1, OLEDSD.3, R15.1; no longer JP2.10
- net VBUS: now also F1.1; no longer L1.1
Other:
- note added: "OLED / Adafruit"
- note added: "OLED / SEEED"
- note added: "OLM-REV-5"
- note added: "uSD"
- note removed: "General"
- note removed: "need to bring up to 3v3?"
- moved on the sheet: CN1, R6

Commit message: changes
Parts:
- removed C29, C30, C31: 10uF, adafruit:C-USC0805K
- removed D3: SCHOTTKY, adafruit:DIODESOD-123
- removed F3: PTCSMD, SparkFun:PTCSMD
- removed R16, R17, R20: 10K, adafruit:R-US_R0805
- removed R18: 10K, rcl:R-EU_R0805
- removed U2: USD-SOCKETMICRO-SD-SOCKET-TAOBAO, SparkFunNew:USD-SOCKETMICRO-SD-SOCKET-TAOBAO
- added C5: 1uF, resistor:C-EUC0805
- added C6: 4.7u, resistor:C-EUC0805
- added C7: .1uF, resistor:C-EUC0805
- added C8, C9: 18pF, resistor:C-EUC0805
- added D2: SCHOTTKY, adafruit:DIODESOD-123
- added F2: PTCSMD, SparkFun:PTCSMD
- added LIPO: MCP73831, SparkFun:MCP73831
- added R13: 10K, adafruit:R-US_R0805
- added R8, R9: 4.7k, adafruit:R-US_R0805
- added RC: 3.3K, rcl:R-EU_R0805
- C10: value 4.7u -> 10uF
- C11, C12: value 100nF -> 10uF; device resistor:C-EUC0402 -> resistor:C-EUC0805
- C13: device adafruit:C-USC0805K -> resistor:C-EUC0805
- C14, C15: value 0.1µ -> 10uF
- C16: value 10u -> 100nF
- C17: value 0.1uF -> 100nF; device rcl:C-USC0805 -> resistor:C-EUC0805
- C18: value .1uF -> 10uF
- C19: value 1uF -> 10uF; device adafruit:C-USC0805K -> adafruit:C-USC0805
- C2: value 18pF -> 1uF; device adafruit:C-USC0805K -> resistor:C-EUC0805
- C20: value 1uF -> .01uF; device adafruit:C-USC0805K -> adafruit:C-USC0805
- C21: value 10uF -> .1uF
- C22: value 10uF -> 0.1uF; device adafruit:C-USC0805 -> rcl:C-USC0805
- C23: value .01uF -> .1uF
- C24, C25: value 10uF -> .1uF; device adafruit:C-USC0805K -> adafruit:C-USC0805
- C26: value .1uF -> 10u; device adafruit:C-USC0805K -> resistor:C-EUC0805
- C27, C28: value 10uF -> 0.1µ; device adafruit:C-USC0805K -> resistor:C-EUC0805
- C3: value 18pF -> 10uF; device adafruit:C-USC0805K -> resistor:C-EUC0805
- C4: value .1uF -> 10uF; device adafruit:C-USC0805 -> resistor:C-EUC0805
- R1: value 22 -> 10K; device adafruit:R-US_R0805 -> rcl:R-EU_R0805
- R10: value 2.32K -> 10K; device rcl:R-EU_R0805 -> adafruit:R-US_R0805
- R11: value 3.3K -> 10K; device rcl:R-EU_R0805 -> adafruit:R-US_R0805
- R14: value 10K -> 1k
- R15: value 10K -> 2.32K; device adafruit:R-US_R0805 -> rcl:R-EU_R0805
- R3: value 1K -> 22
- R4: value 1K -> 470
- R5: value 470 -> 1K
- R6: value 10K -> 1K
- R7: value 1k -> 10K
- U1: value MCP73831 -> USD-SOCKETMICRO-SD-SOCKET-TAOBAO; device SparkFun:MCP73831 -> SparkFunNew:USD-SOCKETMICRO-SD-SOCKET-TAOBAO
- renumbered B2 to B1, DHT22 to DHT1, IC3 to IC2, L2 to L1, R21 to R12, U$1 to BMP1, U6 to LDO, X3 to X1
Connections:
- removed net VDD: BMP1.VDD, C12.1
- removed net VDDIO: BMP1.VDDIO, C11.1
- net +3V3: now also BMP1.VDD, BMP1.VDDIO, C11.1, C12.1, C13.1, C16.1, C19.1, C2.1, C23.1, C25.1, C3.1, R10.1, R11.1, R7.2, R8.2, R9.2, U1.VCC; no longer C20.1, C27.1, C28.1, C30.1, C4.1, R15.2, R16.2, R17.1, R20.1, R5.2, R6.2, U2.VCC
- net +5V: now also C10.1, D2.A, F2.2; no longer C31.1, D1.A, F1.2
- net 3.3V: now also C4.1, C5.1, C7.1, R4.2; no longer C13.1, C19.1, C26.1
- net CHARGE_STAT: now also LIPO.STAT, RC.2; no longer R11.2, U1.STAT
- net D4/A6: now also U1.CS; no longer U2.CS
- net D6*/A8: now also R11.2; no longer R20.2
- net D7/AIN0: now also R10.2; no longer R17.2
- net GND: now also C14.2, C15.2, C23.2, C27.1, C28.1, C5.2, C6.2, C7.2, C8.1, C9.1, LIPO.VSS, R1.1, R13.2, R14.1, R15.1, R5.2, R6.1, U1.GND, U1.SHIELD@1, U1.SHIELD@2, U1.SHIELD@3, U1.SHIELD@4; no longer C14.1, C15.1, C20.2, C27.2, C28.2, C29.2, C30.2, C31.2, R10.1, R14.2, R18.1, R3.1, R4.2, R7.1, U1.VSS, U2.GND, U2.SHIELD@1, U2.SHIELD@2, U2.SHIELD@3, U2.SHIELD@4
- net IO9*/A10: now also R13.1; no longer R14.1
- net MISO: now also U1.DO; no longer U2.DO
- net MOSI: now also U1.DI; no longer U2.DI
- net N$10: now also R4.1; no longer R5.1
- net N$11: now also R5.1; no longer R4.1
- net N$12: now also R6.2; no longer R3.2
- net N$14: now also F1.2; no longer F3.2
- net N$15: now also C27.2; no longer C15.2
- net N$17: now also C26.1; no longer C16.1
- net N$18: now also R15.2; no longer R10.2
- net N$24: now also C20.1; no longer C23.1
- net N$26: now also C20.2; no longer C23.2
- net N$3: now also R3.2; no longer R1.2
- net N$30: now also RC.1; no longer R11.1
- net N$31: now also LIPO.PROG, R1.2; no longer R18.2, U1.PROG
- net N$33: now also D1.A; no longer D3.A
- net N$5: now also R3.1; no longer R1.1
- net N$6: now also R7.1; no longer R6.1
- net N$8: now also C8.2; no longer C2.1
- net N$9: now also C9.2; no longer C3.1
- net SCK: now also U1.SCK; no longer U2.SCK
- net SCK1: now also R14.2; no longer R7.2
- net SCL: now also R8.1; no longer R16.1
- net SDA: now also R9.1; no longer R15.1
- net TCT: now also C28.2; no longer C14.2
- net VBATT: now also C6.1, F1.1, LIPO.VBAT; no longer C10.1, F3.1, U1.VBAT
- net VBUS: now also F2.1; no longer F1.1
- net VCC: now also C14.1, C15.1, D2.C, LIPO.VIN; no longer C25.1, C29.1, D3.C, U1.VIN
Other:
- note added: "Radio"
- note added: "resistors can range from 2.2k to 10k"
- note removed: "I2C pullups"
- moved on the sheet: C10, C11, C12, C13, C14, C15, C16, C17, C18, C19, C2, C20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

Commit message: added schematic and board images
Parts:
- renumbered U1 to MICROSD
Changed lines of the file:
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@@
 <part name="BKOUT" library="SparkFun-Connectors" deviceset="M08" device="LOCK"/>
 <part name="U$2" library="microbuilder" deviceset="GND" device=""/>
-<part name="U1" library="SparkFunNew" deviceset="USD-SOCKET" device="MICRO-SD-SOCKET-TAOBAO" value="USD-SOCKETMICRO-SD-SOCKET-TAOBAO"/>
+<part name="MICROSD" library="SparkFunNew" deviceset="USD-SOCKET" device="MICRO-SD-SOCKET-TAOBAO" value="USD-SOCKETMICRO-SD-SOCKET-TAOBAO"/>
 <part name="GND13" library="SparkFun" deviceset="GND" device=""/>
 <part name="+3V27" library="supply1" deviceset="+3V3" device=""/>
@@
 <instance part="BKOUT" gate="G$1" x="508" y="148.59"/>
 <instance part="U$2" gate="G$1" x="339.09" y="53.34" rot="R90"/>
-<instance part="U1" gate="G$1" x="519.43" y="-90.17"/>
+<instance part="MICROSD" gate="G$1" x="519.43" y="-90.17"/>
 <instance part="GND13" gate="1" x="511.81" y="-110.49"/>
 <instance part="+3V27" gate="G$1" x="510.54" y="-72.39"/>
@@
 </segment>
 <segment>
-<pinref part="U1" gate="G$1" pin="SHIELD@1"/>
-<pinref part="U1" gate="G$1" pin="SHIELD@2"/>
+<pinref part="MICROSD" gate="G$1" pin="SHIELD@1"/>
+<pinref part="MICROSD" gate="G$1" pin="SHIELD@2"/>
 <wire x1="511.81" y1="-100.33" x2="511.81" y2="-102.87" width="0.1524" layer="91"/>
-<pinref part="U1" gate="G$1" pin="SHIELD@3"/>
+<pinref part="MICROSD" gate="G$1" pin="SHIELD@3"/>
 <wire x1="511.81" y1="-102.87" x2="511.81" y2="-105.41" width="0.1524" layer="91"/>
 <junction x="511.81" y="-102.87"/>
-<pinref part="U1" gate="G$1" pin="SHIELD@4"/>
+<pinref part="MICROSD" gate="G$1" pin="SHIELD@4"/>
 <wire x1="511.81" y1="-105.41" x2="511.81" y2="-107.95" width="0.1524" layer="91"/>
 <junction x="511.81" y="-105.41"/>
 <pinref part="GND13" gate="1" pin="GND"/>
 <junction x="511.81" y="-107.95"/>
-<pinref part="U1" gate="G$1" pin="GND"/>
+<pinref part="MICROSD" gate="G$1" pin="GND"/>
 <wire x1="511.81" y1="-90.17" x2="510.54" y2="-90.17" width="0.1524" layer="91"/>
 <wire x1="510.54" y1="-90.17" x2="510.54" y2="-100.33" width="0.1524" layer="91"/>
@@
 </segment>
 <segment>
-<pinref part="U1" gate="G$1" pin="DI"/>
+<pinref part="MICROSD" gate="G$1" pin="DI"/>
 <wire x1="511.81" y1="-82.55" x2="502.92" y2="-82.55" width="0.1524" layer="91"/>
 <label x="504.19" y="-82.55" size="1.778" layer="95"/>
@@
 </segment>
 <segment>
-<pinref part="U1" gate="G$1" pin="DO"/>
+<pinref part="MICROSD" gate="G$1" pin="DO"/>
 <wire x1="511.81" y1="-92.71" x2="502.92" y2="-92.71" width="0.1524" layer="91"/>
 <label x="504.19" y="-92.71" size="1.778" layer="95"/>
@@
 </segment>
 <segment>
-<pinref part="U1" gate="G$1" pin="SCK"/>
+<pinref part="MICROSD" gate="G$1" pin="SCK"/>
 <wire x1="511.81" y1="-87.63" x2="502.92" y2="-87.63" width="0.1524" layer="91"/>
 <label x="504.19" y="-87.63" size="1.778" layer="95"/>
@@
 </segment>
 <segment>
-<pinref part="U1" gate="G$1" pin="VCC"/>
+<pinref part="MICROSD" gate="G$1" pin="VCC"/>
 <wire x1="511.81" y1="-85.09" x2="510.54" y2="-85.09" width="0.1524" layer="91"/>
 <wire x1="510.54" y1="-85.09" x2="510.54" y2="-74.93" width="0.1524" layer="91"/>
@@
 </segment>
 <segment>
-<pinref part="U1" gate="G$1" pin="CS"/>
+<pinref part="MICROSD" gate="G$1" pin="CS"/>
 <wire x1="511.81" y1="-80.01" x2="496.57" y2="-80.01" width="0.1524" layer="91"/>
 <label x="495.3" y="-78.74" size="1.778" layer="95"/>
