File: pcb/eagle/OLMv11.sch (EAGLE design)
At the start: 44 parts, among them IC1 ATMEGA, IC2 MCP1702-33, IC3 ENC28J60SP, J1 1X2-3.5MM, J2 MAGJACK, J3 1X2-3.5MM, J4 1X2-3.5MM, J5 1X2-3.5MM, U1 AM2302, X1 16 MHz, X2 25MHz

Commit message: updated
Parts:
- removed SV3: (no value), con-lstb:MA08-1
- removed U1: AM2302, sensor:AM2302
- added DHT11: (no value), con-lstb:MA04-1
- added LCD1: (no value), con-lstb:MA08-1
- added R11: 330, rcl:R-EU_0204/7
Connections:
- new net AIO1: SV2.2
- new net AIO2: SV2.1
- new net DIO1: SV2.4
- new net DIO2: SV2.3
- new net DIO5: LCD1.8
- new net DIO6: LCD1.7
- new net DIO7: LCD1.6
- new net N$2: R11.1
- new net PWMPIN: LCD1.2
- net +3V3: now also DHT11.1; no longer U1.VDD
- net D0/RX: now also SV2.6
- net D1/TX: now also SV2.5
- net D10/PWM: no longer SV3.1
- net D4: no longer SV3.4
- net D5/PWM: no longer SV3.5
- net D6/PWM: no longer SV3.6
- net DIO-1: now also DHT11.2; no longer U1.DATA
- net GND: now also DHT11.4, LCD1.1, SV2.7; no longer SV3.7, U1.GND
- net MISO/D12: now also LCD1.5
- net MOSI/D11: no longer SV3.3
- net SCK/D13: now also LCD1.4; no longer SV3.2
- net VCC: now also LCD1.3, SV2.8; no longer SV3.8
Other:
- note added: "CE"
- note added: "CLK"
- note added: "DC"
- note added: "DIN"
- note added: "GND"
- note added: "LIGHT"
- note added: "RST"
- note added: "VCC"
