File: pcb/eagle/OLMv11.brd (EAGLE design)
At the start: 100 x 80 mm, 44 parts, among them IC1 ATMEGA, IC2 MCP1702-33, IC3 ENC28J60SP, J1 1X2-3.5MM, J2 MAGJACK, J3 1X2-3.5MM, J4 1X2-3.5MM, J5 1X2-3.5MM, U1 AM2302, X1 16 MHz, X2 25MHz

Commit message: updated
Parts:
- removed SV3: (no value), con-lstb:MA08-1
- removed U1: AM2302, sensor:AM2302
- added DHT11: (no value), con-lstb:MA04-1
- added LCD1: (no value), con-lstb:MA08-1
- added R11: 330, rcl:0204/7
- moved JP5 184.4 mm to (65.8, 40.9), turned to 270 degrees
- moved SV2 169.4 mm to (37.3, 48.8)
- moved J5 168.4 mm to (71.6, 15.7), turned to 90 degrees
- moved J4 166.1 mm to (71.6, 26.4), turned to 90 degrees
- moved JP4 156.8 mm to (65.5, 8.64), turned to 270 degrees
- moved JP3 154.4 mm to (65.5, 18.5), turned to 270 degrees
- moved J1 150.8 mm to (71.6, 5.59), turned to 90 degrees
- moved R3 143.0 mm to (58.2, 7.87)
- moved JP2 140.9 mm to (65.5, 23.9), turned to 90 degrees
- moved SV1 139.7 mm to (69.8, 47.5)
- moved R2 136.2 mm to (58.2, 5.08)
- moved CX2 135.7 mm to (55.9, 23.4)
- moved CX1 126.3 mm to (50.8, 23.1)
- moved R8 120.0 mm to (41.7, 23.9)
- moved R9 117.5 mm to (39.9, 45.0), turned to 180 degrees
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Connections:
- new net AIO1: SV2.2
- new net AIO2: SV2.1
- new net DIO1: SV2.4
- new net DIO2: SV2.3
- new net DIO5: LCD1.8
- new net DIO6: LCD1.7
- new net DIO7: LCD1.6
- new net N$2: R11.1
- new net PWMPIN: LCD1.2
- net +3V3: now also DHT11.1; no longer U1.P$1
- net D0/RX: now also SV2.6
- net D1/TX: now also SV2.5
- net D10/PWM: no longer SV3.1
- net D4: no longer SV3.4
- net D5/PWM: no longer SV3.5
- net D6/PWM: no longer SV3.6
- net DIO-1: now also DHT11.2; no longer U1.P$2
- net GND: now also DHT11.4, LCD1.1, SV2.7; no longer SV3.7, U1.P$4
- net MISO/D12: now also LCD1.5
- net MOSI/D11: no longer SV3.3
- net SCK/D13: now also LCD1.4; no longer SV3.2
- net VCC: now also LCD1.3, SV2.8; no longer SV3.8
Other:
- board size 100 x 80 mm -> 76.1 x 51 mm

Commit message: update
Parts:
- moved D1 2.09 mm to (13.0, 43.7)
- moved R1 1.05 mm to (13.5, 47.8)
Changed lines of the file:
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@@
 <elements>
 <element name="IC1" library="atmega8" package="DIL28-3" value="ATMEGA" x="43.688" y="36.83" rot="R180"/>
-<element name="R1" library="resistor" package="0204/7" value="10k" x="13.716" y="48.768" rot="R180"/>
+<element name="R1" library="resistor" package="0204/7" value="10k" x="13.462" y="47.752" rot="R180"/>
 <element name="IC2" library="JeeLabs" package="TO92" value="MCP1702-33" x="3.556" y="41.91"/>
 <element name="C4" library="resistor" package="E1,8-4" value="10µ" x="22.606" y="41.656" rot="R180"/>
@@
 <element name="R3" library="rcl" package="0204/7" value="1K" x="58.166" y="7.874"/>
 <element name="J2" library="SparkFun" package="MAGJACK" value="MAGJACK" x="0.508" y="17.526" rot="R270"/>
-<element name="D1" library="diode" package="D-5" value="" x="10.922" y="43.18" rot="R180"/>
+<element name="D1" library="diode" package="D-5" value="" x="12.954" y="43.688" rot="R180"/>
 <element name="C2" library="resistor" package="C025-024X044" value="0.1µ" x="59.69" y="44.704"/>
 <element name="R9" library="rcl" package="0204/7" value="10k" x="39.878" y="44.958" rot="R180"/>
@@
 <wire x1="23.495" y1="41.656" x2="39.878" y2="33.02" width="0" layer="19" extent="1-1"/>
 <wire x1="23.114" y1="48.006" x2="23.495" y2="41.656" width="0" layer="19" extent="1-1"/>
-<wire x1="9.906" y1="48.768" x2="23.114" y2="48.006" width="0" layer="19" extent="1-1"/>
-<wire x1="4.826" y1="41.91" x2="9.906" y2="48.768" width="0" layer="19" extent="1-1"/>
+<wire x1="9.652" y1="47.752" x2="23.114" y2="48.006" width="0" layer="19" extent="1-1"/>
+<wire x1="4.826" y1="41.91" x2="9.652" y2="47.752" width="0" layer="19" extent="1-1"/>
 <wire x1="1.778" y1="21.844" x2="4.826" y2="41.91" width="0" layer="19" extent="1-1"/>
 <wire x1="38.862" y1="11.938" x2="39.878" y2="33.02" width="0" layer="19" extent="1-1"/>
@@
 <wire x1="23.114" y1="25.654" x2="2.921" y2="48.26" width="0" layer="19" extent="1-1"/>
 <wire x1="3.556" y1="43.815" x2="23.114" y2="25.654" width="0" layer="19" extent="1-1"/>
-<wire x1="13.462" y1="43.18" x2="3.556" y2="43.815" width="0" layer="19" extent="1-1"/>
+<wire x1="15.494" y1="43.688" x2="3.556" y2="43.815" width="0" layer="19" extent="1-1"/>
 </signal>
 <signal name="D3/PWM">
@@
 <contactref element="SV1" pad="5"/>
 <contactref element="IC3" pad="10"/>
-<wire x1="36.322" y1="19.558" x2="17.526" y2="48.768" width="0" layer="19" extent="1-1"/>
+<wire x1="36.322" y1="19.558" x2="17.272" y2="47.752" width="0" layer="19" extent="1-1"/>
 <wire x1="60.198" y1="40.64" x2="36.322" y2="19.558" width="0" layer="19" extent="1-1"/>
 <wire x1="71.12" y1="46.228" x2="60.198" y2="40.64" width="0" layer="19" extent="1-1"/>
@@
 <contactref element="D1" pad="A"/>
 <contactref element="SV1" pad="2"/>
-<wire x1="66.04" y1="48.768" x2="8.382" y2="43.18" width="0" layer="19" extent="1-1"/>
+<wire x1="66.04" y1="48.768" x2="10.414" y2="43.688" width="0" layer="19" extent="1-1"/>
 </signal>
 <signal name="+3V3">
