File: pcb/eagle/VUSB/open-lab-VUSB-C.sch (EAGLE design)
At the start: 70 parts, among them IC1 ATMEGA328P, IC2 MCP73831, IC4 MCP1700-33, IC5 MCP23008, IC6 MAX31855, IC7 ENC28J60, J1 AYZ0202, Q1 BSS123, Q2 BSS123, Q3 BSS123, X1 USBSMD, X2 32.768kHz, X3 25MHz

Commit message: update
Connections:
- net GND: now also IC5.A0, IC5.A1
Changed lines of the file:
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@@
 <wire x1="-25.4" y1="-63.5" x2="-28.194" y2="-63.5" width="0.1524" layer="91"/>
 <wire x1="-28.194" y1="-63.5" x2="-28.194" y2="-79.502" width="0.1524" layer="91"/>
+<pinref part="IC5" gate="G$1" pin="A1"/>
+<wire x1="-25.4" y1="-60.96" x2="-28.194" y2="-60.96" width="0.1524" layer="91"/>
+<wire x1="-28.194" y1="-60.96" x2="-28.194" y2="-61.214" width="0.1524" layer="91"/>
+<pinref part="IC5" gate="G$1" pin="A0"/>
+<wire x1="-28.194" y1="-61.214" x2="-28.194" y2="-63.5" width="0.1524" layer="91"/>
+<wire x1="-25.4" y1="-58.42" x2="-28.194" y2="-58.42" width="0.1524" layer="91"/>
+<wire x1="-28.194" y1="-58.42" x2="-28.194" y2="-60.96" width="0.1524" layer="91"/>
 </segment>
 <segment>

Commit message: update
Connections:
- net A0: now also SV1.6; no longer Q2.G
- net A1: now also SV1.5; no longer Q1.G
- net A2: now also SV1.4; no longer ETHRESET.1, ETHRESETS.2, IC7.RESET, N5110.1
- net A3: now also SV1.3; no longer RM3.2, RM4.1
- net P0: now also Q2.G; no longer SV1.6
- net P1: now also Q1.G; no longer SV1.5
- net P2: now also ETHRESET.1, ETHRESETS.2, IC7.RESET, N5110.1; no longer SV1.4
- net P3: now also RM3.2, RM4.1; no longer SV1.3
Changed lines of the file:
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@@
 </segment>
 <segment>
-<pinref part="Q2" gate="G$1" pin="G"/>
-<wire x1="167.894" y1="170.434" x2="167.894" y2="172.974" width="0.1524" layer="91"/>
-<label x="167.64" y="173.228" size="1.778" layer="95"/>
+<pinref part="SV1" gate="G$1" pin="6"/>
+<wire x1="43.18" y1="-58.42" x2="41.656" y2="-58.42" width="0.1524" layer="91"/>
+<label x="34.036" y="-58.42" size="1.778" layer="95"/>
 </segment>
 </net>
@@
 </segment>
 <segment>
-<pinref part="IC7" gate="G$1" pin="RESET"/>
-<wire x1="306.578" y1="145.288" x2="292.1" y2="145.288" width="0.1524" layer="91"/>
-<label x="291.338" y="145.796" size="1.778" layer="95"/>
-</segment>
-<segment>
-<pinref part="ETHRESET" gate="A" pin="1"/>
-<wire x1="272.288" y1="163.322" x2="272.288" y2="165.608" width="0.1524" layer="91"/>
-<wire x1="272.288" y1="165.608" x2="274.574" y2="165.608" width="0.1524" layer="91"/>
-<label x="277.876" y="165.862" size="1.778" layer="95"/>
-<wire x1="274.574" y1="165.608" x2="276.86" y2="165.608" width="0.1524" layer="91"/>
-<wire x1="274.574" y1="165.608" x2="274.828" y2="174.752" width="0.1524" layer="91"/>
-<pinref part="ETHRESETS" gate="1" pin="2"/>
-</segment>
-<segment>
-<pinref part="N5110" gate="1" pin="1"/>
-<wire x1="237.236" y1="116.332" x2="243.078" y2="116.332" width="0.1524" layer="91"/>
-<wire x1="243.078" y1="116.332" x2="243.078" y2="116.078" width="0.1524" layer="91"/>
-<label x="243.84" y="115.824" size="1.778" layer="95"/>
+<pinref part="SV1" gate="G$1" pin="4"/>
+<wire x1="43.18" y1="-60.96" x2="41.656" y2="-60.96" width="0.1524" layer="91"/>
+<label x="33.782" y="-60.96" size="1.778" layer="95"/>
 </segment>
 </net>
@@
 </segment>
 <segment>
-<pinref part="RM3" gate="G$1" pin="2"/>
-<pinref part="RM4" gate="G$1" pin="1"/>
-<wire x1="201.93" y1="124.206" x2="201.93" y2="127.762" width="0.1524" layer="91"/>
-<wire x1="201.93" y1="127.762" x2="201.93" y2="135.382" width="0.1524" layer="91"/>
-<wire x1="201.93" y1="127.762" x2="193.802" y2="128.524" width="0.1524" layer="91"/>
-<label x="192.278" y="129.54" size="1.778" layer="95"/>
+<pinref part="SV1" gate="G$1" pin="3"/>
+<wire x1="58.42" y1="-60.96" x2="60.96" y2="-60.96" width="0.1524" layer="91"/>
+<label x="62.484" y="-60.96" size="1.778" layer="95"/>
 </segment>
 </net>
@@
 </segment>
 <segment>
-<pinref part="Q1" gate="G$1" pin="G"/>
-<wire x1="217.424" y1="172.212" x2="217.424" y2="174.752" width="0.1524" layer="91"/>
-<label x="217.17" y="175.006" size="1.778" layer="95"/>
+<pinref part="SV1" gate="G$1" pin="5"/>
+<wire x1="58.42" y1="-58.42" x2="60.96" y2="-58.42" width="0.1524" layer="91"/>
+<label x="62.484" y="-58.42" size="1.778" layer="95"/>
 </segment>
 </net>
@@
 </segment>
 <segment>
-<pinref part="SV1" gate="G$1" pin="3"/>
-<wire x1="58.42" y1="-60.96" x2="60.96" y2="-60.96" width="0.1524" layer="91"/>
-<label x="62.484" y="-60.96" size="1.778" layer="95"/>
+<pinref part="RM3" gate="G$1" pin="2"/>
+<pinref part="RM4" gate="G$1" pin="1"/>
+<wire x1="201.93" y1="124.206" x2="201.93" y2="127.762" width="0.1524" layer="91"/>
+<wire x1="201.93" y1="127.762" x2="201.93" y2="135.382" width="0.1524" layer="91"/>
+<wire x1="201.93" y1="127.762" x2="193.802" y2="128.524" width="0.1524" layer="91"/>
+<label x="192.278" y="129.54" size="1.778" layer="95"/>
 </segment>
 </net>
@@
 </segment>
 <segment>
-<pinref part="SV1" gate="G$1" pin="4"/>
-<wire x1="43.18" y1="-60.96" x2="41.656" y2="-60.96" width="0.1524" layer="91"/>
-<label x="33.782" y="-60.96" size="1.778" layer="95"/>
+<pinref part="IC7" gate="G$1" pin="RESET"/>
+<wire x1="306.578" y1="145.288" x2="292.1" y2="145.288" width="0.1524" layer="91"/>
+<label x="291.338" y="145.796" size="1.778" layer="95"/>
+</segment>
+<segment>
+<pinref part="N5110" gate="1" pin="1"/>
+<wire x1="237.236" y1="116.332" x2="243.078" y2="116.332" width="0.1524" layer="91"/>
+<wire x1="243.078" y1="116.332" x2="243.078" y2="116.078" width="0.1524" layer="91"/>
+<label x="243.84" y="115.824" size="1.778" layer="95"/>
+</segment>
+<segment>
+<pinref part="ETHRESET" gate="A" pin="1"/>
+<wire x1="272.288" y1="163.322" x2="272.288" y2="165.608" width="0.1524" layer="91"/>
+<wire x1="272.288" y1="165.608" x2="274.574" y2="165.608" width="0.1524" layer="91"/>
+<label x="277.876" y="165.862" size="1.778" layer="95"/>
+<wire x1="274.574" y1="165.608" x2="276.86" y2="165.608" width="0.1524" layer="91"/>
+<wire x1="274.574" y1="165.608" x2="274.828" y2="174.752" width="0.1524" layer="91"/>
+<pinref part="ETHRESETS" gate="1" pin="2"/>
 </segment>
 </net>
@@
 </segment>
 <segment>
-<pinref part="SV1" gate="G$1" pin="5"/>
-<wire x1="58.42" y1="-58.42" x2="60.96" y2="-58.42" width="0.1524" layer="91"/>
-<label x="62.484" y="-58.42" size="1.778" layer="95"/>
+<pinref part="Q1" gate="G$1" pin="G"/>
+<wire x1="217.424" y1="172.212" x2="217.424" y2="174.752" width="0.1524" layer="91"/>
+<label x="217.17" y="175.006" size="1.778" layer="95"/>
 </segment>
 </net>
@@
 </segment>
 <segment>
-<pinref part="SV1" gate="G$1" pin="6"/>
-<wire x1="43.18" y1="-58.42" x2="41.656" y2="-58.42" width="0.1524" layer="91"/>
-<label x="34.036" y="-58.42" size="1.778" layer="95"/>
-</segment>
-</net>
+<pinref part="Q2" gate="G$1" pin="G"/>
+<wire x1="167.894" y1="170.434" x2="167.894" y2="172.974" width="0.1524" layer="91"/>
+<label x="167.64" y="173.228" size="1.778" layer="95"/>
+</segment>
+</net>
