File: pcb/eagle/VUSB/open-lab-VUSB-D.brd (EAGLE design)
At the start: 69.5 x 58.4 mm, 72 parts, among them IC1 ATMEGA328P, IC2 MCP73831, IC4 MCP1700-33, IC5 MCP23008, IC6 MAX31855, IC7 ENC28J60, J1 AYZ0202, Q1 BSS123, Q2 BSS123, Q3 BSS123, X1 USBSMD, X2 32.768kHz, X3 25MHz

Commit message: update
Parts:
- moved CEXP1 12.2 mm to (62.0, 15.0), turned to 0 degrees
- moved IC5 4.07 mm to (62.2, 6.86), turned to 270 degrees
- moved RM3 1.55 mm to (33.5, 54.4)
- moved RRST 1.48 mm to (52.8, 14.0), turned to 90 degrees
- moved IC6 1.30 mm to (12.7, 30.0)
- moved Q2 1.14 mm to (53.8, 36.3)
- moved IC2 1.05 mm to (40.9, 3.30)
- moved FB1 1.02 mm to (19.8, 31.5)
- moved REA1 1.02 mm to (27.7, 54.4)
- moved RTCP1 0.92 mm to (19.6, 27.4)
- moved C5 0.92 mm to (43.9, 19.8)
- moved RN3 0.92 mm to (52.8, 31.0)
- moved SV1 0.92 mm to (12.7, 13.5)
- moved RBS 0.80 mm to (26.4, 27.7)
- moved RM4 0.80 mm to (39.1, 54.4)
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
Commit message: update
Parts:
- removed Q1, Q2, Q3: BSS123, transistor-small-signal:SOT23
- added T1, T2, T3: FDN340P, zetex:SOT-23
- moved C6 8.64 mm to (65.5, 54.1)
- moved U$1 4.07 mm to (59.2, 54.4)
- moved RD+ 2.18 mm to (21.3, 12.7)
- moved CTCP 1.80 mm to (16.5, 22.9)
- moved C12 1.30 mm to (49.3, 55.4)
- moved D2 1.27 mm to (11.9, 23.1)
- moved RTCP2 1.08 mm to (20.8, 20.8)
- moved RU 1.05 mm to (27.9, 14.7)
- moved D1 0.76 mm to (9.14, 23.1)
- moved N5110 0.76 mm to (60.5, 28.4)
- moved BTN1 0.57 mm to (66.0, 22.9)
- moved BTN 0.36 mm to (66.0, 34.0)
Connections:
- net LIGHT_LCD: now also T1.2; no longer Q3.3
- net P0: now also T2.3; no longer Q2.1
- net P1: now also T3.3; no longer Q1.1
- net P7: now also T1.3; no longer Q3.1
- net VCC: now also T1.1, T2.1, T3.1; no longer Q1.2, Q2.2, Q3.2
- net V_ETH: now also T3.2; no longer Q1.3
- net V_LCD: now also T2.2; no longer Q2.3
Other:
- board text added: "VUSB-REVD"
- board text removed: "VUSB-REVB"
